File: Hardware/LCMXO/RAM2GS.kicad_pcb (KiCad board)
At the start: 4 copper layers, 67.3 x 48.5 mm, 59 parts, among them J1 Memory Expansion, J2 JTAG, U1 EPM240T100C5N, U10 74LVC1G04GW, U11 AP2127K-1.8TRG1, U2 W9812G6KH-6, U3 60M, U4 74AHCT245PW, U5 74LVC245APW, U6 74LVC245APW, U7 74LVC245APW, U8 AZ1117CH-3.3TRG1, U9 74LVC1G04GW

Commit message: finished MAX, LCMXO, iCE40?
Parts:
- added C29: 2u2, stdpads:C_0603, F.Cu at (91.7, 118.2)
- added R5: DNP, stdpads:R_0805, F.Cu at (62.5, 128.6)
- added RN6: 4x10k, stdpads:R4_0402, F.Cu at (62.9, 126.3)
- added U12: 25F010, stdpads:SOIC-8_3.9mm, F.Cu at (53.1, 127.6)
- U1: value EPM240T100C5N -> LCMXO256-TQFP-100
- U11: value AP2127K-1.8TRG1 -> AP2127K-1.2TRG1
- moved C12 21.8 mm to (79.2, 98.9), turned to 180 degrees
- moved C15 18.1 mm to (75.7, 110.3), turned to 270 degrees
- moved C13 15.7 mm to (86.4, 98.9), turned to 180 degrees
- moved C16 15.0 mm to (95.0, 107.3), turned to 270 degrees
- moved C9 13.4 mm to (84.4, 118.2), turned to 0 degrees
- moved C11 12.5 mm to (75.7, 107.5), turned to 90 degrees
- moved FID4 6.14 mm to (48.5, 124.0)
- moved C14 2.75 mm to (95.0, 110.8), turned to 270 degrees
- turned U1 to 0 degrees
Connections:
- C14 pad 1: +1V8 -> +1V2
- C15 pad 1: +3V3 -> +1V2
- C28 pad 1: +1V8 -> +1V2
- C9 pad 1: +1V8 -> +3V3
- J2 pad 10: GND -> Net-(J2-Pad10)
- J2 pad 3: /TDO -> /TMS
- J2 pad 4: +3V3 -> GND
- J2 pad 5: /TMS -> /TDI
- J2 pad 6: Net-(J2-Pad6) -> +3V3
- J2 pad 7: Net-(J2-Pad7) -> /TDO
- J2 pad 9: /TDI -> Net-(J2-Pad9)
- R4 pad 2: +1V8 -> +1V2
- U1 pad 1: GND -> /Dout0
- U1 pad 10: GND -> +3V3
- U1 pad 100: /R~WE~ -> /RA7
- U1 pad 11: GND -> Net-(U1-Pad11)
- U1 pad 12: /AClk -> GND
- U1 pad 13: +1V8 -> Net-(U1-Pad13)
- U1 pad 14: /BA1 -> /Din2
- U1 pad 15: /RA9 -> /Din1
- U1 pad 16: /RA10 -> /Din3
- U1 pad 17: /RA8 -> /Din5
- U1 pad 18: /RA0 -> /Din4
- U1 pad 19: /RA7 -> /Din7
- U1 pad 2: /DQMH -> /Dout6
- U1 pad 20: /RA1 -> /Din6
- U1 pad 21: /RA6 -> /Din0
- U1 pad 22: /TMS -> /~WE~in
- U1 pad 23: /TDI -> /Ain0
- U1 pad 24: /TCK -> +3V3
- U1 pad 25: /TDO -> GND
- U1 pad 26: /RA4 -> /TMS
- U1 pad 27: /RA3 -> /~CCAS~in
- U1 pad 28: /Dout5 -> /TCK
- U1 pad 29: /RA5 -> /CROWin0
- U1 pad 3: /R~CS~ -> /Dout7
- U1 pad 30: /RA2 -> /CROWin1
- U1 pad 31: +3V3 -> /TDO
- U1 pad 32: GND -> Net-(U1-Pad32)
- U1 pad 33: /Dout0 -> /TDI
- U1 pad 34: /Dout6 -> Net-(U1-Pad34)
- U1 pad 35: /Din2 -> +1V2
- U1 pad 36: /Din1 -> Net-(U1-Pad36)
- U1 pad 37: /Din3 -> /Ain2
- U1 pad 38: /Din5 -> /Ain1
- U1 pad 39: /Din4 -> /PH2in
- U1 pad 4: /R~CAS~ -> /Dout4
- U1 pad 40: /Din7 -> GND
- U1 pad 41: /Din6 -> +3V3
- U1 pad 42: /Din0 -> GND
- U1 pad 43: /Dout7 -> /~CRAS~in
- U1 pad 44: /Dout4 -> /Ain7
- U1 pad 45: +3V3 -> /Ain5
- U1 pad 46: GND -> /Ain4
- U1 pad 47: /Dout3 -> /Ain3
- U1 pad 48: /~WE~in -> Net-(U1-Pad48)
- U1 pad 49: /Ain0 -> /Ain6
- U1 pad 5: /BA0 -> /Dout5
- U1 pad 50: /Ain2 -> /Ain8
- U1 pad 51: /Ain1 -> /Ain9
- U1 pad 52: /PH2in -> Net-(U1-Pad52)
- U1 pad 53: /~CCAS~in -> /S~CS~
- U1 pad 54: /CROWin0 -> Net-(U1-Pad54)
- U1 pad 55: /CROWin1 -> /MISO
- U1 pad 56: /Dout2 -> /MOSI
- U1 pad 57: /Dout1 -> Net-(U1-Pad57)
- U1 pad 58: Net-(U1-Pad58) -> /SCK
- U1 pad 59: +3V3 -> Net-(U1-Pad59)
- U1 pad 6: /R~RAS~ -> /Dout3
- U1 pad 60: GND -> +3V3
- U1 pad 62: Net-(U1-Pad62) -> GND
- U1 pad 63: +1V8 -> Net-(U1-Pad63)
- U1 pad 64: Net-(U1-Pad64) -> /RD0r
- U1 pad 65: GND -> /RD1r
- U1 pad 66: Net-(U1-Pad66) -> /RD3r
- U1 pad 67: /~CRAS~in -> /RD2r
- U1 pad 68: /Ain7 -> /RD5r
- U1 pad 69: /Ain5 -> /RD4r
- U1 pad 7: /RA11 -> /Dout1
- U1 pad 70: /Ain4 -> /RD6r
- U1 pad 71: /Ain3 -> /RD7r
- U1 pad 72: /Ain6 -> /DQML
- U1 pad 73: /Ain8 -> /R~RAS~
- U1 pad 74: /Ain9 -> +3V3
- U1 pad 75: Net-(U1-Pad75) -> GND
- U1 pad 76: Net-(U1-Pad76) -> /R~WE~
- U1 pad 77: /MISO -> /R~CS~
- U1 pad 78: Net-(U1-Pad78) -> /DQMH
- U1 pad 79: GND -> /BA0
- U1 pad 8: /CKE -> /Dout2
- U1 pad 80: +3V3 -> /R~CAS~
- U1 pad 81: Net-(U1-Pad81) -> /RA11
- U1 pad 82: Net-(U1-Pad82) -> /CKE
- U1 pad 83: /MOSI -> /BA1
- U1 pad 84: Net-(U1-Pad84) -> GND
- U1 pad 85: /SCK -> /RA9
- U1 pad 86: Net-(U1-Pad86) -> /AClk
- U1 pad 87: /S~CS~ -> /RA10
- U1 pad 88: Net-(U1-Pad88) -> +3V3
- U1 pad 89: /RD2r -> /RA1
- U1 pad 9: +3V3 -> Net-(U1-Pad9)
- U1 pad 90: /RD1r -> +1V2
- U1 pad 91: /RD5r -> /RA6
- U1 pad 92: /RD4r -> +3V3
- U1 pad 94: +3V3 -> /RA2
- U1 pad 95: /RD6r -> /RA5
- U1 pad 96: /RD0r -> /RA8
- U1 pad 97: /RD7r -> /RA3
- U1 pad 98: /DQML -> /RA0
- U1 pad 99: /RD3r -> /RA4
- U11 pad 5: +1V8 -> +1V2
Routing:
- net +1V8: track 143.8 -> 0.00 mm, vias 8 -> 0
- net +1V2: track 0.00 -> 105.8 mm, vias 0 -> 9
- net /MOSI: track 0.00 -> 92.6 mm, vias 0 -> 3
- net /SCK: track 0.00 -> 90.2 mm, vias 0 -> 3
- net /MISO: track 0.00 -> 82.5 mm, vias 0 -> 2
- net /S~CS~: track 0.00 -> 81.2 mm, vias 0 -> 2
- net /TMS: track 59.1 -> 30.3 mm, vias 3 -> 2
- net /Dout1: track 21.7 -> 7.57 mm, vias 2 -> 0
- net /Dout2: track 19.8 -> 7.51 mm, vias 2 -> 0
- net +5V: track 181.7 -> 193.9 mm
- net /TDI: track 39.0 -> 27.0 mm
- net /~HLD~: track 0.00 -> 11.6 mm, vias 0 -> 1
- net /Ain2: track 7.82 -> 19.1 mm, vias 0 -> 2
- net /Dout3: track 18.7 -> 7.63 mm, vias 2 -> 0
- net /RD0r: track 13.2 -> 23.8 mm
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- added copper zone on F.Cu, net +1V2
- removed copper zone on F.Cu, net +1V8

Commit message: almost done
Parts:
- U1: value LCMXO256-TQFP-100 -> LCMXO256C-3TN100C
Connections:
- U1 pad 48: Net-(U1-Pad48) -> GND
Routing:
- net GND: track 179.1 -> 180.2 mm, vias 219 -> 220
- net Net-(U1-Pad48): track 1.11 -> 0.00 mm, vias 1 -> 0
- net /TDO: track 31.1 -> 30.4 mm

Commit message: more
Parts:
- U1: value LCMXO256C-3TN100C -> LCMXO640-TQFP-100
Connections:
- U1 pad 29: /CROWin0 -> +3V3
- U1 pad 30: /CROWin1 -> GND
- U1 pad 32: Net-(U1-Pad32) -> /CROWin0
- U1 pad 34: Net-(U1-Pad34) -> /CROWin1
- U1 pad 48: GND -> +3V3
- U1 pad 61: Net-(U1-Pad61) -> /DQML
- U1 pad 63: Net-(U1-Pad63) -> /BA0
- U1 pad 72: /DQML -> /R~WE~
- U1 pad 76: /R~WE~ -> /DQMH
- U1 pad 78: /DQMH -> /R~CAS~
- U1 pad 79: /BA0 -> /RA11
- U1 pad 80: /R~CAS~ -> +3V3
- U1 pad 81: /RA11 -> GND
Routing:
- net /DQML: track 34.4 -> 43.0 mm
- net /BA0: track 34.3 -> 42.9 mm
- net +3V3: track 269.7 -> 276.8 mm, vias 103 -> 108
- net /R~WE~: track 29.0 -> 34.5 mm
- net /CROWin1: track 12.7 -> 16.4 mm
- net GND: track 180.2 -> 183.8 mm, vias 220 -> 221
- net /CROWin0: track 11.9 -> 15.0 mm, vias 0 -> 2
- net /Ain2: track 19.1 -> 20.6 mm
- net /Ain1: track 19.9 -> 21.4 mm
- net /PH2in: track 20.1 -> 21.4 mm
- net /DQMH: track 17.3 -> 18.5 mm
- net /R~CAS~: track 28.3 -> 29.5 mm
- net /RA11: track 22.7 -> 23.7 mm
- net /TCK: track 30.5 -> 31.2 mm
- net /TDO: track 30.4 -> 31.1 mm

Commit message: Generated gerbers and documenation PDFs
Parts:
- removed RN1, RN2, RN3, RN4, RN5: 4x33, stdpads:R4_0402
- removed RN6: 4x10k, stdpads:R4_0402
- added C30: 15p, stdpads:C_0603, F.Cu at (95.0, 99.5)
- added D1: White, stdpads:LED_0805, F.Cu at (71.3, 102.7)
- added R6: 47, stdpads:R_0603, F.Cu at (70.5, 108.0)
- added R7: 47, stdpads:R_0603, F.Cu at (73.2, 108.0)
- added R8: 180, stdpads:R_0805, F.Cu at (71.3, 104.6)
- J1: value Memory Expansion -> IIgs RAM Exp.
- R3: value 100 -> 47; footprint stdpads:R_0805 -> stdpads:R_0603
- R5: value DNP -> 47; footprint stdpads:R_0805 -> stdpads:R_0603
- U1: value LCMXO640-TQFP-100 -> LCMXO256-TN100
- moved R5 46.6 mm to (97.8, 98.2), turned to 45 degrees
- moved R3 26.9 mm to (96.8, 115.8), turned to 270 degrees
Connections:
- J2 pad 1: /TCK -> /TCKr
- R3 pad 1: Net-(R3-Pad1) -> /~CRAS~in
- R5 pad 1: /~HLD~ -> /TCK
- R5 pad 2: GND -> /TCKr
- U1 pad 57: Net-(U1-Pad57) -> /LED
- U1 pad 64: /RD0r -> /RD0
- U1 pad 65: /RD1r -> /RD1
- U1 pad 66: /RD3r -> /RD2
- U1 pad 67: /RD2r -> /RD3
- U1 pad 68: /RD5r -> /RD4
- U1 pad 69: /RD4r -> /RD5
- U1 pad 70: /RD6r -> /RD6
- U1 pad 71: /RD7r -> /RD7
- U12 pad 7: /~HLD~ -> +3V3
- U4 pad 19: Net-(R3-Pad2) -> Net-(U4-Pad19)
- U7 pad 11: Net-(RN5-Pad4) -> /Ain9
- U7 pad 12: Net-(RN5-Pad3) -> /Ain8
- U7 pad 13: Net-(RN5-Pad2) -> /Ain6
- U7 pad 14: Net-(RN5-Pad1) -> /Ain3
- U7 pad 15: Net-(RN4-Pad4) -> /Ain4
- U7 pad 16: Net-(RN4-Pad3) -> /Ain5
- U7 pad 17: Net-(RN4-Pad2) -> /Ain7
- U7 pad 18: Net-(RN4-Pad1) -> Net-(R3-Pad2)
- U9 pad 4: Net-(R3-Pad1) -> Net-(U4-Pad19)
Routing:
- net /RD0r: track 23.8 -> 0.00 mm, vias 2 -> 0
- net /RD0: track 18.6 -> 41.1 mm
- net /RD3r: track 22.1 -> 0.00 mm, vias 2 -> 0
- net /RD5r: track 22.1 -> 0.00 mm, vias 2 -> 0
- net /LED: track 0.00 -> 21.5 mm
- net /RD6r: track 21.1 -> 0.00 mm, vias 2 -> 0
- net /RD2: track 19.4 -> 40.4 mm
- net /RD1r: track 20.2 -> 0.00 mm, vias 2 -> 0
- net /RD4: track 20.0 -> 39.8 mm
- net /RD4r: track 19.6 -> 0.00 mm, vias 2 -> 0
- net /RD2r: track 19.2 -> 0.00 mm, vias 2 -> 0
- net /RD1: track 19.3 -> 38.4 mm
- net /RD6: track 20.2 -> 38.7 mm
- net /RD3: track 19.5 -> 37.9 mm
- net /RD7r: track 18.3 -> 0.00 mm, vias 2 -> 0
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- added copper zone on F.Cu, net +3V3
Other:
- board text added: "D20B"
