File: Hardware/LCMXO/RAM2GS.kicad_pcb (KiCad board)
At the start: 4 copper layers, 67.3 x 48.5 mm, 64 parts, among them J1 IIgs RAM Exp., J2 JTAG, U1 LCMXO256C-3TN100C, U10 74LVC1G04GW, U11 AP2127K-1.2TRG1, U12 25F010, U2 W9812G6KH-6, U3 60M, U4 74AHCT245PW, U5 74LVC245APW, U6 74LVC245APW, U7 74LVC245APW, U8 AZ1117CH-3.3TRG1, U9 74LVC1G04GW

Commit message: RC D.2.3
Connections:
- U2 pad 40: (no net) -> unconnected-(U2-NC-Pad40)
Other:
- board text added: "D23B"
- board text removed: "D22B"
