File: Hardware/LCMXO/RAM2GS.sch (KiCad schematic (older format))
At the start: 59 parts, among them J1 Memory Expansion, J2 JTAG, U1 EPM240T100C5N, U10 74LVC1G04GW, U11 AP2127K-1.8TRG1, U2 W9812G6KH-6, U3 60M, U4 74AHCT245PW, U5 74LVC245APW, U6 74LVC245APW, U7 74LVC245APW, U8 AZ1117CH-3.3TRG1, U9 74LVC1G04GW

Commit message: finished MAX, LCMXO, iCE40?
Parts:
- removed U1: EPM240T100C5N, stdpads:TQFP-100_14x14mm_P0.5mm, symbol GW_PLD:5M240ZT100
- removed U11: AP2127K-1.8TRG1, stdpads:SOT-23-5, symbol Regulator_Linear:AP2127K-1.8
- added C29: 2u2, stdpads:C_0603, symbol Device:C_Small
- added R5: DNP, stdpads:R_0805, symbol Device:R_Small
- added RN6: 4x10k, stdpads:R4_0402, symbol Device:R_Pack04
- added U1: LCMXO256-TQFP-100, stdpads:TQFP-100_14x14mm_P0.5mm, symbol GW_PLD:LCMXO256-TQFP-100
- added U11: AP2127K-1.2TRG1, stdpads:SOT-23-5, symbol Regulator_Linear:AP2127K-1.2
- added U12: 25F010, stdpads:SOIC-8_3.9mm, symbol GW_RAM:SPIFlash-SO-8
Connections:
- net labels added: +1V2, ~HLD~
- net labels removed: +1V8
- wire segments 91 -> 101
- no-connect marks 23 -> 10
Other:
- moved on the sheet: C10, C14, C15, C27, C9

Commit message: almost done
Parts:
- U1: value LCMXO256-TQFP-100 -> LCMXO256C-3TN100C; Mfg. Part Numbers Lattice LCMXO256C-3TN100C -> Lattice LCMXO256C-3TN100C, Lattice LCMXO256C-4TN100C, Latti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
- U2: Mfg. Part Numbers Winbond W9812G6KH-6 Winbond W9812G6KH-6I, Winbond W9825G6KH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 -> Winbond W9812G6KH-6, Winbond W9812G6KH-6I, Winbond W9825G6K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
- U3: Notes Most 60-62.5 MHz crystal oscillator or silicon oscillator i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 -> Most 60-62.5 MHz 3.3V crystal oscillator or silicon oscilla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
Connections:
- net GND: now also U1.48 (~SLEEP~)
- no-connect marks 10 -> 22
Other:
- moved on the sheet: C28, R4
Changed lines of the file:
@@
 L power:+3V3 #PWR0133
 U 1 1 5E9850F8
-P 2050 3850
-F 0 "#PWR0133" H 2050 3700 50  0001 C CNN
-F 1 "+3V3" H 2050 4000 50  0000 C CNN
-F 2 "" H 2050 3850 50  0001 C CNN
-F 3 "" H 2050 3850 50  0001 C CNN
-	1    2050 3850
+P 2150 3850
+F 0 "#PWR0133" H 2150 3700 50  0001 C CNN
+F 1 "+3V3" H 2150 4000 50  0000 C CNN
+F 2 "" H 2150 3850 50  0001 C CNN
+F 3 "" H 2150 3850 50  0001 C CNN
+	1    2150 3850
 	1    0    0    -1
 $EndComp
@@
 L power:+5V #PWR0134
 U 1 1 5E9856CC
-P 1050 3850
-F 0 "#PWR0134" H 1050 3700 50  0001 C CNN
-F 1 "+5V" H 1050 4000 50  0000 C CNN
-F 2 "" H 1050 3850 50  0001 C CNN
-F 3 "" H 1050 3850 50  0001 C CNN
-	1    1050 3850
+P 950 3850
+F 0 "#PWR0134" H 950 3700 50  0001 C CNN
+F 1 "+5V" H 950 4000 50  0000 C CNN
+F 2 "" H 950 3850 50  0001 C CNN
+F 3 "" H 950 3850 50  0001 C CNN
+	1    950  3850
 	-1   0    0    -1
 $EndComp
@@
 F 3 "" H 9400 2650 50  0001 C CNN
 F 4 "C62379" H 9400 2900 50  0001 C CNN "LCSC Part"
-F 5 "Winbond W9812G6KH-6 Winbond W9812G6KH-6I, Winbond W9825G6KH-6, Winbond W9825G6KH-6I, ISSI IS42S16160J-6TL, ISSI IS42S16160J-6TLI, Micron MT48LC16M16A2P-6A :G, Micron MT48LC16M16A2P-6A IT:G" H 9400 2900 50  0001 C CNN "Mfg. Part Numbers"
+F 5 "Winbond W9812G6KH-6, Winbond W9812G6KH-6I, Winbond W9825G6KH-6, Winbond W9825G6KH-6I, ISSI IS42S16160J-6TL, ISSI IS42S16160J-6TLI, Micron MT48LC16M16A2P-6A :G, Micron MT48LC16M16A2P-6A IT:G" H 9400 2900 50  0001 C CNN "Mfg. Part Numbers"
 F 6 "Most 166 MHz 128/256 Mbit SDRAM is acceptable." H 9400 2900 50  0001 C CNN "Notes"
 	1    9400 2900
@@
 F 4 "C26255" H 9950 5050 50  0001 C CNN "LCSC Part"
 F 5 "SiTime SIT1602AI-82-33E-60.000000Y, Shenzhen SCTF S7D60.000000B20F30T, Taiten OCETGLJTNF-60MHZ" H 9950 5050 50  0001 C CNN "Mfg. Part Numbers"
-F 6 "Most 60-62.5 MHz crystal oscillator or silicon oscillator is acceptable. Do not use crystal resonator or ceramic resonator." H 9950 5050 50  0001 C CNN "Notes"
+F 6 "Most 60-62.5 MHz 3.3V crystal oscillator or silicon oscillator is acceptable. Do not use crystal resonator or ceramic resonator." H 9950 5050 50  0001 C CNN "Notes"
 	1    9950 5050
 	-1   0    0    -1
@@
 $EndComp
 Wire Wire Line
-	2050 3850 1850 3850
-Wire Wire Line
-	1050 3850 1250 3850
+	2150 3850 1950 3850
+Wire Wire Line
+	950  3850 1250 3850
 Connection ~ 2650 6950
 Connection ~ 2250 7350
@@
 $EndComp
 Wire Wire Line
-	1250 4650 1050 4650
-Wire Wire Line
-	1050 4650 1050 4550
-Connection ~ 1050 3850
-Wire Wire Line
-	1250 4550 1050 4550
-Connection ~ 1050 4550
-Wire Wire Line
-	1050 4550 1050 3850
+	1250 4650 950  4650
+Wire Wire Line
+	950  4650 950  4550
+Connection ~ 950  3850
+Wire Wire Line
+	1250 4550 950  4550
+Connection ~ 950  4550
+Wire Wire Line
+	950  4550 950  3850
 $Comp
 L power:GND #PWR0161
@@
 L power:+1V2 #PWR0162
 U 1 1 86F3BCA1
-P 2050 4550
-F 0 "#PWR0162" H 2050 4400 50  0001 C CNN
-F 1 "+1V2" H 2050 4700 50  0000 C CNN
-F 2 "" H 2050 4550 50  0001 C CNN
-F 3 "" H 2050 4550 50  0001 C CNN
-	1    2050 4550
-	1    0    0    -1
-$EndComp
-Wire Wire Line
-	2050 4550 1850 4550
+P 2150 4550
+F 0 "#PWR0162" H 2150 4400 50  0001 C CNN
+F 1 "+1V2" H 2150 4700 50  0000 C CNN
+F 2 "" H 2150 4550 50  0001 C CNN
+F 3 "" H 2150 4550 50  0001 C CNN
+	1    2150 4550
+	1    0    0    -1
+$EndComp
+Wire Wire Line
+	2150 4550 1950 4550
 $Comp
 L Device:R_Small R4
 U 1 1 86F45A5D
-P 1850 4200
-F 0 "R4" H 1791 4246 50  0000 R CNN
-F 1 "0" H 1791 4155 50  0000 R CNN
-F 2 "stdpads:R_0805" H 1850 4200 50  0001 C CNN
-F 3 "" H 1850 4200 50  0001 C CNN
-F 4 "C17477" H 1850 4200 50  0001 C CNN "LCSC Part"
-F 5 "Any manufacturer's part is acceptable." H 1850 4200 50  0001 C CNN "Notes"
-F 6 "Uniroyal 0805W8F0000T5E" H 1850 4200 50  0001 C CNN "Mfg. Part Numbers"
-	1    1850 4200
-	-1   0    0    -1
-$EndComp
-Wire Wire Line
-	1850 4100 1850 3850
-Connection ~ 1850 3850
-Wire Wire Line
-	1850 4550 1850 4300
-Connection ~ 1850 4550
+P 1950 4200
+F 0 "R4" H 1891 4246 50  0000 R CNN
+F 1 "0" H 1891 4155 50  0000 R CNN
+F 2 "stdpads:R_0805" H 1950 4200 50  0001 C CNN
+F 3 "" H 1950 4200 50  0001 C CNN
+F 4 "C17477" H 1950 4200 50  0001 C CNN "LCSC Part"
+F 5 "Any manufacturer's part is acceptable." H 1950 4200 50  0001 C CNN "Notes"
+F 6 "Uniroyal 0805W8F0000T5E" H 1950 4200 50  0001 C CNN "Mfg. Part Numbers"
+	1    1950 4200
+	-1   0    0    -1
+$EndComp
 $Comp
 L Device:C_Small C28
 U 1 1 86F60831
-P 2050 4650
-F 0 "C28" H 2142 4696 50  0000 L CNN
-F 1 "2u2" H 2142 4605 50  0000 L CNN
-F 2 "stdpads:C_0603" H 2050 4650 50  0001 C CNN
-F 3 "" H 2050 4650 50  0001 C CNN
-F 4 "C23630" H 2050 4650 50  0001 C CNN "LCSC Part"
-F 5 "10V or higher. Any manufacturer's part is acceptable but Samsung, Murata, Yageo preferred." H 2050 4650 50  0001 C CNN "Notes"
-F 6 "Samsung CL10A225KO8NNNC" H 2050 4650 50  0001 C CNN "Mfg. Part Numbers"
-	1    2050 4650
-	1    0    0    -1
-$EndComp
-Connection ~ 2050 4550
-Wire Wire Line
-	2050 4750 2050 4950
-Wire Wire Line
-	2050 4950 1550 4950
+P 2150 4650
+F 0 "C28" H 2242 4696 50  0000 L CNN
+F 1 "2u2" H 2242 4605 50  0000 L CNN
+F 2 "stdpads:C_0603" H 2150 4650 50  0001 C CNN
+F 3 "" H 2150 4650 50  0001 C CNN
+F 4 "C23630" H 2150 4650 50  0001 C CNN "LCSC Part"
+F 5 "10V or higher. Any manufacturer's part is acceptable but Samsung, Murata, Yageo preferred." H 2150 4650 50  0001 C CNN "Notes"
+F 6 "Samsung CL10A225KO8NNNC" H 2150 4650 50  0001 C CNN "Mfg. Part Numbers"
+	1    2150 4650
+	1    0    0    -1
+$EndComp
+Connection ~ 2150 4550
+Wire Wire Line
+	2150 4750 2150 4950
+Wire Wire Line
+	2150 4950 1550 4950
 Connection ~ 1550 4950
 $Comp
@@
 P 6300 3300
 F 0 "U1" H 6300 3350 50  0000 C CNN
-F 1 "LCMXO256-TQFP-100" H 6300 3250 40  0000 C CNN
+F 1 "LCMXO256C-3TN100C" H 6300 3250 40  0000 C CNN
 F 2 "stdpads:TQFP-100_14x14mm_P0.5mm" H 6300 3200 40  0001 C CNN
 F 3 "" H 6300 3400 50  0001 C CNN
 F 4 "C1521848" H 6300 3300 50  0001 C CNN "LCSC Part"
-F 5 "Lattice LCMXO256C-3TN100C" H 6300 3300 50  0001 C CNN "Mfg. Part Numbers"
+F 5 "Lattice LCMXO256C-3TN100C, Lattice LCMXO256C-4TN100C, Lattice LCMXO256C-5TN100C" H 6300 3300 50  0001 C CNN "Mfg. Part Numbers"
 	1    6300 3300
 	1    0    0    -1
 $EndComp
+NoConn ~ 5350 2000
+NoConn ~ 5350 2100
+NoConn ~ 5350 2200
+NoConn ~ 5350 3700
+NoConn ~ 5350 3800
+NoConn ~ 5350 3900
+NoConn ~ 7250 4400
+NoConn ~ 7250 4500
+NoConn ~ 7250 4600
+NoConn ~ 7250 4800
+NoConn ~ 7250 5100
+NoConn ~ 7250 5300
+Wire Wire Line
+	1950 4300 1950 4550
+Connection ~ 1950 4550
+Wire Wire Line
+	1950 4550 1850 4550
+Wire Wire Line
+	1950 4100 1950 3850
+Connection ~ 1950 3850
+Wire Wire Line
+	1950 3850 1850 3850
+$Comp
+L power:GND #PWR?
+U 1 1 60E703CE
+P 7550 1200
+F 0 "#PWR?" H 7550 950 50  0001 C CNN
+F 1 "GND" H 7550 1050 50  0000 C CNN
+F 2 "" H 7550 1200 50  0001 C CNN
+F 3 "" H 7550 1200 50  0001 C CNN
+	1    7550 1200
+	-1   0    0    -1
+$EndComp
+Wire Wire Line
+	7550 1200 7250 1200
 $EndSCHEMATC

Commit message: more
Parts:
- removed U1: LCMXO256C-3TN100C, stdpads:TQFP-100_14x14mm_P0.5mm, symbol GW_PLD:LCMXO256-TQFP-100
- added U1: LCMXO640-TQFP-100, stdpads:TQFP-100, symbol GW_PLD:LCMXO640-TQFP-100
Connections:
- net +1V2: now also U1.35 (Vcc), U1.90 (Vcc)
- net +3V3: now also U1.10 (VccIO3), U1.24 (VccIO3), U1.29 (VccIO2), U1.41 (VccIO2), U1.48 (~SLEEP~), U1.60 (VccIO1), U1.74 (VccIO1), U1.80 (VccIO0), U1.88 (VccAUX), U1.92 (VccIO0)
- net AClk: now also U1.86 (PT5B/PCLK0_0)
- net Ain0: now also U1.23 (PL11C)
- net Ain1: now also U1.38 (PB6B/PCLK2_0)
- net Ain2: now also U1.37 (PB5D)
- net Ain3: now also U1.47 (PB9C)
- net Ain4: now also U1.46 (PB9A)
- net Ain5: now also U1.45 (PB8D)
- net Ain6: now also U1.49 (PB9D)
- net Ain7: now also U1.44 (PB8C)
- net Ain8: now also U1.50 (PB9F)
- net Ain9: now also U1.51 (PR11D)
- net BA0: now also U1.63 (PR7B)
- net BA1: now also U1.83 (PT7A)
- net CKE: now also U1.82 (PT7E)
- net CROWin0: now also U1.32 (PB4C)
- net CROWin1: now also U1.34 (PB4E)
- net DQMH: now also U1.76 (PR9F)
- net DQML: now also U1.61 (PR9B)
- net Din0: now also U1.21 (PL10C)
- net Din1: now also U1.15 (PL7B)
- net Din2: now also U1.14 (PL5B/~GSRN~)
- net Din3: now also U1.16 (PL8C/TSALL)
- net Din4: now also U1.18 (PL9A)
- net Din5: now also U1.17 (PL8D)
- net Din6: now also U1.20 (PL10A)
- net Din7: now also U1.19 (PL9C)
- net Dout0: now also U1.1 (PL2A)
- net Dout1: now also U1.7 (PL3C)
- net Dout2: now also U1.8 (PL3D)
- net Dout3: now also U1.6 (PL3B)
- net Dout4: now also U1.4 (PL2D)
- net Dout5: now also U1.5 (PL3A)
- net Dout6: now also U1.2 (PL2C)
- net Dout7: now also U1.3 (PL2B)
- net GND: now also U1.12 (GNDIO3), U1.25 (GNDIO3), U1.30 (GNDIO2), U1.40 (GND), U1.42 (GNDIO2), U1.62 (GNDIO1), U1.75 (GNDIO1), U1.81 (GNDIO0), U1.84 (GND), U1.93 (GNDIO0)
- net MISO: now also U1.55 (PR10D)
- net MOSI: now also U1.56 (PR10C)
- net PH2in: now also U1.39 (PB6C)
- net RA0: now also U1.98 (PT2B)
- net RA1: now also U1.89 (PT4F)
- net RA10: now also U1.87 (PT5A)
- net RA11: now also U1.79 (PT9A)
- net RA2: now also U1.94 (PT3B)
- net RA3: now also U1.97 (PT2E)
- net RA4: now also U1.99 (PT2C)
- net RA5: now also U1.95 (PT3A)
- net RA6: now also U1.91 (PT3F)
- net RA7: now also U1.100 (PT2A)
- net RA8: now also U1.96 (PT2F)
- net RA9: now also U1.85 (PT6B/PCLK0_1)
- net RD0r: now also U1.64 (PR6C)
- net RD1r: now also U1.65 (PR6B)
- net RD2r: now also U1.67 (PR5B)
- net RD3r: now also U1.66 (PR5D)
- net RD4r: now also U1.69 (PR4B)
- net RD5r: now also U1.68 (PR4D)
- net RD6r: now also U1.70 (PR3D)
- net RD7r: now also U1.71 (PR3B)
- net R~CAS~: now also U1.78 (PT9C)
- net R~CS~: now also U1.77 (PT9E)
- net R~RAS~: now also U1.73 (PR2B)
- net R~WE~: now also U1.72 (PR2D)
- net SCK: now also U1.58 (PR10A)
- net S~CS~: now also U1.53 (PR11C)
- net TCK: now also U1.28 (TCK)
- net TDI: now also U1.33 (TDI)
- net TDO: now also U1.31 (TDO)
- net TMS: now also U1.26 (TMS)
- net ~CCAS~in: now also U1.27 (PL2C)
- net ~CRAS~in: now also U1.43 (PB8B)
- net ~WE~in: now also U1.22 (PL11A)
- no-connect marks 22 -> 14
Changed lines of the file:
@@
 Text Label 8900 3900 2    50   ~ 0
 RClk
-Text Label 7250 2300 0    50   ~ 0
+Text Label 7450 2300 0    50   ~ 0
 AClk
 Wire Wire Line
@@
 L power:GND #PWR0136
 U 1 1 5E9DF65F
-P 6600 5700
-F 0 "#PWR0136" H 6600 5450 50  0001 C CNN
-F 1 "GND" H 6600 5550 50  0000 C CNN
-F 2 "" H 6600 5700 50  0001 C CNN
-F 3 "" H 6600 5700 50  0001 C CNN
-	1    6600 5700
+P 6800 5700
+F 0 "#PWR0136" H 6800 5450 50  0001 C CNN
+F 1 "GND" H 6800 5550 50  0000 C CNN
+F 2 "" H 6800 5700 50  0001 C CNN
+F 3 "" H 6800 5700 50  0001 C CNN
+	1    6800 5700
 	-1   0    0    -1
 $EndComp
@@
 Text Label 5350 3200 2    50   ~ 0
 Ain0
-Text Label 5350 3600 2    50   ~ 0
+Text Label 5350 3800 2    50   ~ 0
 CROWin1
-Text Label 5350 3500 2    50   ~ 0
+Text Label 5350 3700 2    50   ~ 0
 CROWin0
 Text Label 5350 3400 2    50   ~ 0
@@
 Text Label 5350 4900 2    50   ~ 0
 Ain8
-Text Label 7250 3000 0    50   ~ 0
+Text Label 7450 3200 0    50   ~ 0
 DQMH
-Text Label 7250 2800 0    50   ~ 0
+Text Label 7450 3000 0    50   ~ 0
 R~CAS~
-Text Label 7250 2600 0    50   ~ 0
+Text Label 7450 2600 0    50   ~ 0
 CKE
-Text Label 7250 3400 0    50   ~ 0
+Text Label 7450 3400 0    50   ~ 0
 R~RAS~
-Text Label 7250 3100 0    50   ~ 0
+Text Label 7450 3100 0    50   ~ 0
 R~CS~
-Text Label 7250 2900 0    50   ~ 0
+Text Label 7450 4400 0    50   ~ 0
 BA0
-Text Label 7250 2700 0    50   ~ 0
+Text Label 7450 2900 0    50   ~ 0
 RA11
-Text Label 7250 2500 0    50   ~ 0
+Text Label 7450 2500 0    50   ~ 0
 BA1
-Text Label 7250 2400 0    50   ~ 0
+Text Label 7450 2400 0    50   ~ 0
 RA9
-Text Label 7250 2200 0    50   ~ 0
+Text Label 7450 2200 0    50   ~ 0
 RA10
-Text Label 7250 1700 0    50   ~ 0
+Text Label 7450 1700 0    50   ~ 0
 RA8
-Text Label 7250 1500 0    50   ~ 0
+Text Label 7450 1500 0    50   ~ 0
 RA0
-Text Label 7250 1300 0    50   ~ 0
+Text Label 7450 1300 0    50   ~ 0
 RA7
-Text Label 7250 2100 0    50   ~ 0
+Text Label 7450 2100 0    50   ~ 0
 RA1
-Text Label 7250 2000 0    50   ~ 0
+Text Label 7450 2000 0    50   ~ 0
 RA6
-Text Label 7250 1900 0    50   ~ 0
+Text Label 7450 1900 0    50   ~ 0
 RA2
-Text Label 7250 1600 0    50   ~ 0
+Text Label 7450 1600 0    50   ~ 0
 RA3
-Text Label 7250 1400 0    50   ~ 0
+Text Label 7450 1400 0    50   ~ 0
 RA4
-Text Label 7250 1800 0    50   ~ 0
+Text Label 7450 1800 0    50   ~ 0
 RA5
 $Comp
@@
 	0    1    -1   0
 $EndComp
-Text Label 7250 5200 0    50   ~ 0
+Text Label 7450 5200 0    50   ~ 0
 S~CS~
-Text Label 7250 4700 0    50   ~ 0
+Text Label 7450 4700 0    50   ~ 0
 SCK
-Text Label 7250 4900 0    50   ~ 0
+Text Label 7450 4900 0    50   ~ 0
 MOSI
-Text Label 7250 5000 0    50   ~ 0
+Text Label 7450 5000 0    50   ~ 0
 MISO
 Text Label 5350 4100 2    50   ~ 0
@@
 Text Label 5350 4000 2    50   ~ 0
 Ain2
-Text Label 7250 3200 0    50   ~ 0
+Text Label 7450 3500 0    50   ~ 0
 R~WE~
-Text Label 7250 3500 0    50   ~ 0
+Text Label 7450 4500 0    50   ~ 0
 DQML
-Text Label 7250 4300 0    50   ~ 0
+Text Label 7450 4300 0    50   ~ 0
 RD0r
-Text Label 7250 3600 0    50   ~ 0
+Text Label 7450 3600 0    50   ~ 0
 RD7r
-Text Label 7250 3700 0    50   ~ 0
+Text Label 7450 3700 0    50   ~ 0
 RD6r
-Text Label 7250 3900 0    50   ~ 0
+Text Label 7450 3900 0    50   ~ 0
 RD5r
-Text Label 7250 3800 0    50   ~ 0
+Text Label 7450 3800 0    50   ~ 0
 RD4r
-Text Label 7250 4100 0    50   ~ 0
+Text Label 7450 4100 0    50   ~ 0
 RD3r
-Text Label 7250 4000 0    50   ~ 0
+Text Label 7450 4000 0    50   ~ 0
 RD2r
-Text Label 7250 4200 0    50   ~ 0
+Text Label 7450 4200 0    50   ~ 0
 RD1r
 Text Label 5350 5400 2    50   ~ 0
@@
 $EndComp
 Connection ~ 2250 6750
-Text Label 7250 5400 0    50   ~ 0
+Text Label 7450 5400 0    50   ~ 0
 Ain9
-Connection ~ 6200 5700
-Connection ~ 6600 5700
-Connection ~ 6400 5700
-Connection ~ 6200 900
-Wire Wire Line
-	6300 5700 6400 5700
-Wire Wire Line
-	6200 5700 6300 5700
-Connection ~ 6300 5700
-Wire Wire Line
-	6300 900  6400 900
-Wire Wire Line
-	6200 900  6300 900
-Connection ~ 6300 900
-Wire Wire Line
-	6100 5700 6200 5700
-Connection ~ 6100 5700
-Wire Wire Line
-	6100 900  6200 900
-Connection ~ 6100 900
-Wire Wire Line
-	6500 5700 6600 5700
-Wire Wire Line
-	6400 5700 6500 5700
-Connection ~ 6500 5700
 Wire Wire Line
 	6600 900  6700 900
-Wire Wire Line
-	6000 900  6100 900
-Wire Wire Line
-	5900 900  6000 900
-Connection ~ 6000 900
-Wire Wire Line
-	6000 5700 6100 5700
-Wire Wire Line
-	5900 5700 6000 5700
-Connection ~ 6000 5700
-Connection ~ 5900 900
 Wire Wire Line
 	4000 6950 4000 7050
 Connection ~ 4000 6950
-Connection ~ 6400 900
-Wire Wire Line
-	6400 900  6500 900
 $Comp
 L power:+1V2 #PWR0150
 U 1 1 8715E9C7
-P 6600 900
-F 0 "#PWR0150" H 6600 750 50  0001 C CNN
-F 1 "+1V2" H 6600 1050 50  0000 C CNN
-F 2 "" H 6600 900 50  0001 C CNN
-F 3 "" H 6600 900 50  0001 C CNN
-	1    6600 900
-	1    0    0    -1
-$EndComp
-Connection ~ 6600 900
+P 6800 900
+F 0 "#PWR0150" H 6800 750 50  0001 C CNN
+F 1 "+1V2" H 6800 1050 50  0000 C CNN
+F 2 "" H 6800 900 50  0001 C CNN
+F 3 "" H 6800 900 50  0001 C CNN
+	1    6800 900
+	1    0    0    -1
+$EndComp
 Wire Wire Line
 	1450 6950 1850 6950
@@
 	0    1    1    0
 $EndComp
-$Comp
-L GW_PLD:LCMXO256-TQFP-100 U1
-U 1 1 86DF1B11
-P 6300 3300
-F 0 "U1" H 6300 3350 50  0000 C CNN
-F 1 "LCMXO256C-3TN100C" H 6300 3250 40  0000 C CNN
-F 2 "stdpads:TQFP-100_14x14mm_P0.5mm" H 6300 3200 40  0001 C CNN
-F 3 "" H 6300 3400 50  0001 C CNN
-F 4 "C1521848" H 6300 3300 50  0001 C CNN "LCSC Part"
-F 5 "Lattice LCMXO256C-3TN100C, Lattice LCMXO256C-4TN100C, Lattice LCMXO256C-5TN100C" H 6300 3300 50  0001 C CNN "Mfg. Part Numbers"
-	1    6300 3300
-	1    0    0    -1
-$EndComp
 NoConn ~ 5350 2000
 NoConn ~ 5350 2100
 NoConn ~ 5350 2200
-NoConn ~ 5350 3700
-NoConn ~ 5350 3800
 NoConn ~ 5350 3900
-NoConn ~ 7250 4400
-NoConn ~ 7250 4500
-NoConn ~ 7250 4600
-NoConn ~ 7250 4800
-NoConn ~ 7250 5100
-NoConn ~ 7250 5300
 Wire Wire Line
 	1950 4300 1950 4550
@@
 	1950 3850 1850 3850
 $Comp
-L power:GND #PWR?
-U 1 1 60E703CE
-P 7550 1200
-F 0 "#PWR?" H 7550 950 50  0001 C CNN
-F 1 "GND" H 7550 1050 50  0000 C CNN
-F 2 "" H 7550 1200 50  0001 C CNN
-F 3 "" H 7550 1200 50  0001 C CNN
-	1    7550 1200
-	-1   0    0    -1
-$EndComp
-Wire Wire Line
-	7550 1200 7250 1200
+L power:+3V3 #PWR0168
+U 1 1 626AF4E6
+P 7450 1200
+F 0 "#PWR0168" H 7450 1050 50  0001 C CNN
+F 1 "+3V3" H 7450 1350 50  0000 C CNN
+F 2 "" H 7450 1200 50  0001 C CNN
+F 3 "" H 7450 1200 50  0001 C CNN
+	1    7450 1200
+	1    0    0    -1
+$EndComp
+Wire Wire Line
+	5900 900  6000 900
+Wire Wire Line
+	5900 5700 6000 5700
+$Comp
+L GW_PLD:LCMXO640-TQFP-100 U1
+U 1 1 62C26D47
+P 6400 3300
+F 0 "U1" H 6400 811 50  0000 C CNN
+F 1 "LCMXO640-TQFP-100" H 6400 727 40  0000 C CNN
+F 2 "stdpads:TQFP-100" H 6400 3200 40  0001 C CNN
+F 3 "" H 6400 3400 50  0001 C CNN
+	1    6400 3300
+	1    0    0    -1
+$EndComp
+Connection ~ 5900 900
+Wire Wire Line
+	6800 5700 6700 5700
+Connection ~ 6800 5700
+Connection ~ 6000 5700
+Connection ~ 6100 5700
+Wire Wire Line
+	6100 5700 6000 5700
+Connection ~ 6200 5700
+Wire Wire Line
+	6200 5700 6100 5700
+Connection ~ 6300 5700
+Wire Wire Line
+	6300 5700 6200 5700
+Connection ~ 6400 5700
+Wire Wire Line
+	6400 5700 6300 5700
+Connection ~ 6500 5700
+Wire Wire Line
+	6500 5700 6400 5700
+Connection ~ 6600 5700
+Wire Wire Line
+	6600 5700 6500 5700
+Connection ~ 6700 5700
+Wire Wire Line
+	6700 5700 6600 5700
+Wire Wire Line
+	6500 900  6400 900
+Connection ~ 6000 900
+Connection ~ 6100 900
+Wire Wire Line
+	6100 900  6000 900
+Connection ~ 6200 900
+Wire Wire Line
+	6200 900  6100 900
+Connection ~ 6300 900
+Wire Wire Line
+	6300 900  6200 900
+Connection ~ 6400 900
+Wire Wire Line
+	6400 900  6300 900
+Wire Wire Line
+	6600 900  6500 900
+Connection ~ 6600 900
+Connection ~ 6500 900
+Wire Wire Line
+	6800 900  6900 900
+Connection ~ 6800 900
 $EndSCHEMATC

Commit message: Generated gerbers and documenation PDFs
Parts:
- removed RN1, RN2, RN3, RN4, RN5: 4x33, stdpads:R4_0402, symbol Device:R_Pack04
- removed RN6: 4x10k, stdpads:R4_0402, symbol Device:R_Pack04
- added C30: 15p, stdpads:C_0603, symbol Device:C_Small
- added D1: White, stdpads:LED_0805, symbol Device:LED_Small_ALT
- added R6, R7: 47, stdpads:R_0603, symbol Device:R_Small
- added R8: 180, stdpads:R_0805, symbol Device:R_Small
- J1: value Memory Expansion -> IIgs RAM Exp.
- R3: value 100 -> 47; footprint stdpads:R_0805 -> stdpads:R_0603; LCSC Part C17408 -> C23182; Mfg. Part Numbers Uniroyal 0805W8F1000T5E -> Uniroyal 0603WAF470JT5E
- R5: value DNP -> 47; footprint stdpads:R_0805 -> stdpads:R_0603; LCSC Part (none) -> C23182; Mfg. Part Numbers (none) -> Uniroyal 0603WAF470JT5E; Notes (none) -> Any manufacturer's part is acceptable.
- U1: value LCMXO640-TQFP-100 -> LCMXO256-TN100; footprint stdpads:TQFP-100 -> stdpads:TQFP-100_14x14mm_P0.5mm; LCSC Part (none) -> C1550734; Mfg. Part Numbers (none) -> Lattice LCMXO256C-3TN100C, Lattice LCMXO256C-4TN100C, Latti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
- U10, U9: Mfg. Part Numbers NXP 74LVC1G04GW, TI SN74LVC1G04DCK -> NXP 74LVC1G04GW, TI SN74LVC1G04DCK, NXP 74AHC1G04GW, TI SN7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; Notes (none) -> Most 74LVC1G04 or 74AHC1G04 in SOT-353 package is acceptabl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
- U11: Notes (none) -> Most 1.2V regulator in SOT-23-5 package is acceptable.
- U12: LCSC Part (none) -> C2687406; Notes Most SPI flash in SOIC-8 (3.9mm / 150 mil width) package is acceptale. -> Most SPI flash in SOIC-8 (3.9mm / 150 mil width) package is acceptable.
- U2: Notes Most 166 MHz 128/256 Mbit SDRAM is acceptable. -> Most 166 MHz 128/256 Mbit x16 SDRAM is acceptable.
- U4: Mfg. Part Numbers NXP 74AHCT245PW, TI SN74AHCT245PW -> NXP 74AHCT245PW, NXP 74AHCT245APW, TI SN74AHCT245PW; Notes (none) -> Most 74AHCT245 in TSSOP-20 package is acceptable.
- U5, U6, U7: Mfg. Part Numbers NXP 74LVC245APW, TI SN74LVC245APW -> NXP 74LVC245APW, TI SN74LVC245APW, NXP 74AHC245PW, NXP 74AH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; Notes (none) -> Most 74LVC245 or 74AHC245 in TSSOP-20 package is acceptable.
Connections:
- net RD0r is gone; now on net RD0: U1.64 (PR6C)
- net RD1r is gone; now on net RD1: U1.65 (PR6B)
- net RD2r is gone; now on net RD3: U1.67 (PR5B)
- net RD3r is gone; now on net RD2: U1.66 (PR5D)
- net RD4r is gone; now on net RD5: U1.69 (PR4B)
- net RD5r is gone; now on net RD4: U1.68 (PR4D)
- net RD6r is gone; now on net RD6: U1.70 (PR3D)
- net RD7r is gone; now on net RD7: U1.71 (PR3B)
- net +3V3: now also U12.7 (~HLD~/IO3), R8.2
- net AClk: now also R7.2
- net Ain3: now also U7.14 (B4)
- net Ain4: now also U7.15 (B3)
- net Ain5: now also U7.16 (B2)
- net Ain6: now also U7.13 (B5)
- net Ain7: now also U7.17 (B1)
- net Ain8: now also U7.12 (B6)
- net Ain9: now also U7.11 (B7)
- net GND: now also C30.2; no longer R5.2
- net RClk: now also R6.2
- net TCK: now also R5.1, C30.1; no longer J2.1 (Pin_1)
- net ~CRAS~in: now also R3.1
- net at U4.19 (~OE~): now also U9.4 (Y); no longer R3.2
- net at U7.18 (B0): now also R3.2
- net at U10.4 (Y): now also R6.1, R7.1
- net LED: now reaches U1.57 (PR10B)
- net LED: now also D1.1 (K)
- removed net ~HLD~: R5.1, U12.7 (~HLD~/IO3)
- new net: D1.2 (A), R8.1
- new net TCKr: J2.1 (Pin_1), R5.2
- no-connect marks 14 -> 10
Other:
- moved on the sheet: J2, R1, R2
