File: Hardware/LCMXO/RAM2GS.kicad_sch (KiCad schematic)
At the start: 62 parts, among them J1 IIgs RAM Exp., J2 JTAG, U1 LCMXO256-TN100, U10 74LVC1G04GW, U11 AP2127K-1.2TRG1, U12 25F010, U2 W9812G6KH-6, U3 60M, U4 74AHCT245PW, U5 74LVC245APW, U6 74LVC245APW, U7 74LVC245APW, U8 AZ1117CH-3.3TRG1, U9 74LVC1G04GW

Commit message: RC 2.2
Parts:
- C1, C2, C26, C3, C4: Mfg. Part Numbers Samsung CL21A106KAYNNNE -> (none); Notes 10V or higher. Any manufacturer's part is acceptable but Sa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 -> (none)
- C10, C11, C12, C13, C14, C15, C16, C17, C18, C19, C20, C21, C22, C23, C24, C25, C27, C28, C29, C5, C6, C7, C8, C9: Mfg. Part Numbers Samsung CL10A225KO8NNNC -> (none); Notes 10V or higher. Any manufacturer's part is acceptable but Sa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 -> (none)
- C30: LCSC Part C1644 -> C1653; Mfg. Part Numbers Samsung CL10C150JB8NNNC -> (none); Notes 10V or higher. Any manufacturer's part is acceptable but Sa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 -> (none)
- D1: LCSC Part (none) -> C284932; Notes Any manufacturer's part is acceptable. -> (none)
- FID1, FID2, FID3, FID4: Notes DNP - SMT vision system fiducial -> (none)
- H1, H2, H4, H5: Notes DNP - mounting hole for solder paste printing -> (none)
- H3: Notes DNP - mounting hole -> (none)
- J1: Notes DNP - edge connector -> (none)
- J2: footprint Connector:Tag-Connect_TC2050-IDC-FP_2x05_P1.27mm_Vertical -> stdpads:Tag-Connect_TC2050-IDC-FP_2x05_P1.27mm_Vertical; Notes DNP - test pad connector -> (none)
- R1, R2: Mfg. Part Numbers Uniroyal 0805W8F2202T5E -> (none); Notes Any manufacturer's part is acceptable. -> (none)
- R3, R5, R6, R7: Mfg. Part Numbers Uniroyal 0603WAF470JT5E -> (none); Notes Any manufacturer's part is acceptable. -> (none)
- R4: Mfg. Part Numbers Uniroyal 0805W8F0000T5E -> (none); Notes Any manufacturer's part is acceptable. -> (none)
- R8: Mfg. Part Numbers Uniroyal 0805W8F2200T5E -> (none); Notes Any manufacturer's part is acceptable. -> (none)
- U1: value LCMXO256-TN100 -> LCMXO256C-4TN100C; Mfg. Part Numbers Lattice LCMXO256C-3TN100C, Lattice LCMXO256C-4TN100C, Latti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 -> (none)
- U10, U9: Mfg. Part Numbers NXP 74LVC1G04GW, TI SN74LVC1G04DCK, NXP 74AHC1G04GW, TI SN7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 -> (none); Notes Most 74LVC1G04 or 74AHC1G04 in SOT-353 package is acceptabl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 -> (none)
- U11: Mfg. Part Numbers Diodes AP2127K-1.2TRG1, Torex XC6228D122VR -> (none); Notes Most 1.2V regulator in SOT-23-5 package is acceptable. -> (none)
- U12: LCSC Part C2687406 -> C19617; Mfg. Part Numbers Zetta ZD25WD20BTIGT, Adesto AT25SF081-SSHD, Winbond W25X20C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 -> (none); Notes Most SPI flash in SOIC-8 (3.9mm / 150 mil width) package is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 -> (none)
- U2: Mfg. Part Numbers Winbond W9812G6KH-6, Winbond W9812G6KH-6I, Winbond W9825G6K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 -> (none); Notes Most 166 MHz 128/256 Mbit x16 SDRAM is acceptable. -> (none)
- U3: Mfg. Part Numbers SiTime SIT1602AI-82-33E-60.000000Y, Shenzhen SCTF S7D60.000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 -> (none); Notes Most 60-62.5 MHz 3.3V crystal oscillator or silicon oscilla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 -> (none)
- U4: Mfg. Part Numbers NXP 74AHCT245PW, NXP 74AHCT245APW, TI SN74AHCT245PW -> (none); Notes Most 74AHCT245 in TSSOP-20 package is acceptable. -> (none)
- U5, U6, U7: Mfg. Part Numbers NXP 74LVC245APW, TI SN74LVC245APW, NXP 74AHC245PW, NXP 74AH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 -> (none); Notes Most 74LVC245 or 74AHC245 in TSSOP-20 package is acceptable. -> (none)
- U8: Mfg. Part Numbers Diodes AZ1117CH-3.3TRG1, Diodes AZ1117EH-3.3TRG1 -> (none); Notes Most 1117-type 3.3V regulator in SOT-223 package is accepta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 -> (none)
Connections:
- net +5V: no longer J1.11 (Pin_11)
- new net 5VC: J1.11 (Pin_11)

Commit message: RC
Parts:
- C30: value 15p -> 22p
- U1: value LCMXO256C-4TN100C -> LCMXO256C-3TN100C; LCSC Part C1550734 -> C1521848
Connections:
- no-connect marks 9 -> 12
Changed lines of the file:
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@@
   (junction (at 57.15 161.29) (diameter 0) (color 0 0 0 0)
   )
+  (no_connect (at 189.23 116.84))
   (no_connect (at 135.89 53.34))
   (no_connect (at 135.89 99.06))
@@
   (no_connect (at 123.19 24.13))
   (no_connect (at 81.28 186.69))
+  (no_connect (at 189.23 134.62))
   (no_connect (at 93.98 186.69))
   (no_connect (at 135.89 55.88))
+  (no_connect (at 189.23 129.54))
   (no_connect (at 135.89 50.8))
   (wire (pts (xy 67.31 161.29) (xy 57.15 161.29))
@@
       (effects (font (size 1.27 1.27)))
     )
-    (property "Value" "LCMXO256C-4TN100C" (at 162.56 83.82 0)
+    (property "Value" "LCMXO256C-3TN100C" (at 162.56 83.82 0)
       (effects (font (size 1.016 1.016)))
     )
@@
       (effects (font (size 1.27 1.27)) hide)
     )
-    (property "LCSC Part" "C1550734" (at 162.56 83.82 0)
+    (property "LCSC Part" "C1521848" (at 162.56 83.82 0)
       (effects (font (size 1.27 1.27)) hide)
     )
@@
       (effects (font (size 1.27 1.27)) (justify left))
     )
-    (property "Value" "15p" (at 111.5568 187.833 0)
+    (property "Value" "22p" (at 111.5568 187.833 0)
       (effects (font (size 1.27 1.27)) (justify left))
     )

Commit message: 2.2
Parts:
- H1, H2, H3, H4, H5: value (none) -> (none)

Commit message: RC D.2.3
Parts:
- H1, H2, H3, H4, H5: value (none) -> ~
Connections:
- no-connect marks 12 -> 13
Changed lines of the file:
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@@
 	(title_block
 		(title "GW4201D (RAM2GS II) - LCMXO256 / LCMXO640")
-		(date "2024-04-24")
-		(rev "2.2")
+		(date "2025-02-14")
+		(rev "2.3")
 		(company "Garrett's Workshop")
 	)
@@
 		(at 135.89 50.8)
 	)
+	(no_connect
+		(at 250.19 93.98)
+	)
 	(wire
 		(pts
@@
 		(pin "9"
 		)
+		(pin "40"
+		)
 		(instances
 			(project "RAM2GS"
@@
 			)
 		)
-		(property "Value" ""
+		(property "Value" "~"
 			(at 69.85 88.646 0)
 			(effects
@@
 			)
 		)
-		(property "Value" ""
+		(property "Value" "~"
 			(at 57.15 87.376 0)
 			(effects
@@
 			)
 		)
-		(property "Value" ""
+		(property "Value" "~"
 			(at 31.75 87.376 0)
 			(effects
@@
 			)
 		)
-		(property "Value" ""
+		(property "Value" "~"
 			(at 44.45 87.376 0)
 			(effects
@@
 			)
 		)
-		(property "Value" ""
+		(property "Value" "~"
 			(at 19.05 87.376 0)
 			(effects
