File: Hardware/LCMXO2/RAM2GS.sch (KiCad schematic (older format))
At the start: 61 parts, among them J1 Memory Expansion, J2 JTAG, U1 LCMXO256-TQFP-100, U10 74LVC1G04GW, U11 SPIFlash-SON-8-1EP, U12 AP2127K-1.2, U2 W9812G6KH-6, U3 60M, U4 74AHCT245PW, U5 74LVC245APW, U6 74LVC245APW, U7 74LVC245APW, U8 AZ1117CH-3.3, U9 74LVC1G04GW

Commit message: finished MAX, LCMXO, iCE40?
Parts:
- removed U1: LCMXO256-TQFP-100, stdpads:TQFP-100_14x14mm_P0.5mm, symbol GW_PLD:LCMXO256-TQFP-100
- removed U11: SPIFlash-SON-8-1EP, stdpads:SON-8-1EP_3x2mm_P0.5mm_EP0.25x1.65mm, symbol GW_RAM:SPIFlash-SON-8-1EP
- added U1: LCMXO2-640-TQFP-100, stdpads:TQFP-100_14x14mm_P0.5mm, symbol GW_PLD:LCMXO2-640-TQFP-100
- C1, C2, C26, C3, C4: Mfg. Part Numbers (none) -> Samsung CL21A106KAYNNNE; Notes 10V or higher -> 10V or higher. Any manufacturer's part is acceptable but Sa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
- C10, C11, C12, C13, C14, C15, C16, C17, C18, C19, C20, C21, C22, C23, C24, C25, C27, C28, C29, C5, C6, C7, C8, C9: Mfg. Part Numbers (none) -> Samsung CL10A225KO8NNNC; Notes 10V or higher -> 10V or higher. Any manufacturer's part is acceptable but Sa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
- R1, R2: Mfg. Part Numbers (none) -> Uniroyal 0805W8F2202T5E; Notes Any manufacturer's part is acceptable -> Any manufacturer's part is acceptable.
- R3: Mfg. Part Numbers (none) -> Uniroyal 0805W8F1000T5E; Notes Any manufacturer's part is acceptable -> Any manufacturer's part is acceptable.
- R4: Mfg. Part Numbers (none) -> Uniroyal 0805W8F0000T5E; Notes Any manufacturer's part is acceptable -> Any manufacturer's part is acceptable.
- RN1, RN2, RN3, RN4, RN5: Mfg. Part Numbers (none) -> Uniroyal 4D02WGJ0330TCE; Notes Any manufacturer's part is acceptable -> Any manufacturer's part is acceptable.
- U10, U9: Mfg. Part Numbers NXP 74LVC1G04GW TI SN74LVC1G04DCK -> NXP 74LVC1G04GW, TI SN74LVC1G04DCK
- U11: renamed from U12; value AP2127K-1.2 -> AP2127K-1.2TRG1; LCSC Part (none) -> C151376; Mfg. Part Numbers (none) -> Diodes AP2127K-1.2TRG1, Torex XC6228D122VR
- U2: Notes Most 166 MHz 128/256 Mbit SDRAM will work -> Most 166 MHz 128/256 Mbit SDRAM is acceptable.
- U3: Mfg. Part Numbers SiTime SIT1602AI-82-33E-60.000000Y -> SiTime SIT1602AI-82-33E-60.000000Y, Shenzhen SCTF S7D60.000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; Notes Most 60-64 MHz crystal oscillator or silicon oscillator wil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 -> Most 60-62.5 MHz crystal oscillator or silicon oscillator i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
- U4: Mfg. Part Numbers NXP 74AHCT245PW TI SN74AHCT245PW -> NXP 74AHCT245PW, TI SN74AHCT245PW
- U5, U6, U7: Mfg. Part Numbers NXP 74LVC245APW TI SN74LVC245APW -> NXP 74LVC245APW, TI SN74LVC245APW
- U8: value AZ1117CH-3.3 -> AZ1117CH-3.3TRG1; Mfg. Part Numbers Diodes AZ1117CH-3.3TR1G Diodes AZ1117EH-3.3TR1G -> Diodes AZ1117CH-3.3TRG1, Diodes AZ1117EH-3.3TRG1; Notes (none) -> Most 1117-type 3.3V regulator in SOT-223 package is accepta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
Connections:
- net labels removed: D2, D3, MISO, MOSI, SCK, S~CS~
- wire segments 94 -> 95
Other:
- moved on the sheet: C28, FID1, FID2, FID3, FID4, H1, H2, H3, H4, H5, R4, RN1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

Commit message: almost done
Parts:
- removed R1, R2: 22k, stdpads:R_0805, symbol Device:R_Small
- added RN7: 4x10k, stdpads:R4_0402, symbol Device:R_Pack04
- U1: value LCMXO2-640-TQFP-100 -> LCMXO2-640HC-4TG100C; symbol GW_PLD:LCMXO2-640-TQFP-100 -> GW_PLD:LCMXO2-640-TG100; LCSC Part (none) -> C1519051; Mfg. Part Numbers (none) -> Lattice LCMXO2-640HC-4TG100C, Lattice LCMXO2-640HC-5TG100C,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
- U2: Mfg. Part Numbers Winbond W9812G6KH-6 Winbond W9812G6KH-6I, Winbond W9825G6KH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 -> Winbond W9812G6KH-6, Winbond W9812G6KH-6I, Winbond W9825G6K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
- U3: Notes Most 60-62.5 MHz crystal oscillator or silicon oscillator i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 -> Most 60-62.5 MHz 3.3V crystal oscillator or silicon oscilla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
Connections:
- net +3V3: now also RN7.2 (R2.1), RN7.3 (R3.1), RN7.4 (R4.1)
- net AClk: now also U1.62 (PCLKC1_0/PR5D); no longer U1.78 (PT11A)
- net Ain0: now also U1.14 (PL5C); no longer U1.28 (PB4B)
- net Ain1: now also U1.12 (PL5A/PCLKT3_1); no longer U1.36 (PB10A)
- net Ain2: now also U1.13 (PL5B/PCLKC3_1); no longer U1.35 (PB6D/PCLKC_0)
- net Ain3: now also U1.21 (PL7B/PCLKC3_0); no longer U1.42 (PB12C)
- net Ain4: now also U1.20 (PL7A/PCLKT3_0); no longer U1.41 (PB12B)
- net Ain5: now also U1.19 (PL6D); no longer U1.40 (PB12A)
- net Ain6: now also U1.24 (PL7C); no longer U1.43 (PB12D)
- net Ain7: now also U1.18 (PL6C); no longer U1.39 (PB10D/PCLKC2_1)
- net Ain8: now also U1.25 (PL7D); no longer U1.45 (PB14A)
- net Ain9: now also U1.32 (PB6B/SO/SPISO); no longer U1.51 (PR7D)
- net BA0: now also U1.58 (PR6C); no longer U1.68 (PR3B)
- net BA1: now also U1.60 (PR6A); no longer U1.74 (PR2B)
- net CKE: now also U1.53 (PR7B); no longer U1.71 (PR2C)
- net CROWin0: now also U1.10 (PL3D); no longer U1.30 (PB4D)
- net CROWin1: now also U1.16 (PL6A); no longer U1.34 (PB6C/PCLKT2_0)
- net DQMH: now also U1.51 (PR7D); no longer U1.67 (PR3C)
- net DQML: now also U1.48 (PB14C/SN); no longer U1.63 (PCLKT1_0/PR5C)
- net Din0: now also U1.3 (PL2C/PCLKT3_2); no longer U1.24 (PL7C)
- net Din1: now also U1.96 (PT6D); no longer U1.16 (PL6A)
- net Din2: now also U1.88 (PT9A/PCLKT0_1); no longer U1.15 (PL5D)
- net Din3: now also U1.97 (PT6C); no longer U1.17 (PL6B)
- net Din4: now also U1.99 (PT6A); no longer U1.19 (PL6D)
- net Din5: now also U1.98 (PT6B); no longer U1.18 (PL6C)
- net Din6: now also U1.2 (PL2B); no longer U1.21 (PL7B/PCLKC3_0)
- net Din7: now also U1.1 (PL2A); no longer U1.20 (PL7A/PCLKT3_0)
- net Dout1: now also U1.86 (SCL/PCLKT0_0/PT9C); no longer U1.9 (PL3C)
- net Dout2: now also U1.87 (PT9B/PCLKC0_1); no longer U1.10 (PL3D)
- net Dout3: now also U1.85 (SDA/PCLKC0_0/PT9D); no longer U1.8 (PL3B)
- net Dout4: now also U1.83 (PT10B); no longer U1.4 (PL2D/PCLKC3_2)
- net Dout5: now also U1.84 (PT10A); no longer U1.7 (PL3A)
- net Dout6: now also U1.78 (PT11A); no longer U1.2 (PL2B)
- net Dout7: now also U1.82 (~JTAGEN~/PT10C); no longer U1.3 (PL2C/PCLKT3_2)
- net GND: now also RN7.1 (R1.1)
- net PH2in: now also U1.8 (PL3B); no longer U1.37 (PB10B)
- net RA0: now also U1.66 (PR3D); no longer U1.97 (PT6C)
- net RA1: now also U1.67 (PR3C); no longer U1.84 (PT10A)
- net RA10: now also U1.64 (PR5B); no longer U1.83 (PT10B)
- net RA11: now also U1.59 (PR6B); no longer U1.70 (PR2D)
- net RA2: now also U1.69 (PR3A); no longer U1.86 (SCL/PCLKT0_0/PT9C)
- net RA3: now also U1.71 (PR2C); no longer U1.96 (PT6D)
- net RA4: now also U1.74 (PR2B); no longer U1.98 (PT6B)
- net RA5: now also U1.70 (PR2D); no longer U1.87 (PT9B/PCLKC0_1)
- net RA6: now also U1.68 (PR3B); no longer U1.85 (SDA/PCLKC0_0/PT9D)
- net RA7: now also U1.75 (PR2A); no longer U1.99 (PT6A)
- net RA8: now also U1.65 (PR5A); no longer U1.88 (PT9A/PCLKT0_1)
- net RA9: now also U1.63 (PCLKT1_0/PR5C); no longer U1.75 (PR2A)
- net RD0r: now also U1.36 (PB10A); no longer U1.52 (PR7C)
- net RD1r: now also U1.37 (PB10B); no longer U1.53 (PR7B)
- net RD2r: now also U1.39 (PB10D/PCLKC2_1); no longer U1.57 (PR6D)
- net RD3r: now also U1.38 (PB10C/PCLKT2_1); no longer U1.54 (PR7A)
- net RD4r: now also U1.41 (PB12B); no longer U1.59 (PR6B)
- net RD5r: now also U1.40 (PB12A); no longer U1.58 (PR6C)
- net RD6r: now also U1.42 (PB12C); no longer U1.60 (PR6A)
- net RD7r: now also U1.43 (PB12D); no longer U1.62 (PCLKC1_0/PR5D)
- net R~CAS~: now also U1.52 (PR7C); no longer U1.69 (PR3A)
- net R~CS~: now also U1.57 (PR6D); no longer U1.66 (PR3D)
- net R~RAS~: now also U1.54 (PR7A); no longer U1.64 (PR5B)
- net R~WE~: now also U1.49 (PB14D/SI/SISPI); no longer U1.65 (PR5A)
- net TCK: now also RN7.8 (R1.2)
- net ~CCAS~in: now also U1.9 (PL3C); no longer U1.29 (PB4C)
- net ~CRAS~in: now also U1.17 (PL6B); no longer U1.38 (PB10C/PCLKT2_1)
- net ~WE~in: now also U1.15 (PL5D); no longer U1.25 (PL7D)
- net DONE: now reaches U1.76 (DONE/PT11D)
- net DONE: now also U4.18 (B0), RN7.6 (R3.2)
- net ~INIT~: now reaches U1.77 (~INIT~/PT11C)
- net ~INIT~: now also RN7.7 (R2.2)
- net ~PROG~: now reaches U1.81 (~PROGRAM~/PT10D)
- net ~PROG~: now also RN7.5 (R4.2)
- removed net Dout0: U1.1 (PL2A), U4.18 (B0)
- no-connect marks 10 -> 21
Other:
- moved on the sheet: C28, R4

Commit message: more
Parts:
- added R1: 2k2, stdpads:R_0603, symbol Device:R_Small
- RN7: LCSC Part C25501 -> C25725; Mfg. Part Numbers Uniroyal 4D02WGJ0330TCE -> Uniroyal 4D02WGJ0103TCE
Connections:
- net Dout7: now also R1.1
- net GND: now also R1.2
Changed lines of the file:
@@
 Wire Wire Line
 	5600 6650 5600 6550
-Text Label 7550 3200 0    50   ~ 0
-DONE
 Wire Wire Line
 	7250 3200 7550 3200
@@
 F 2 "stdpads:R4_0402" V 5675 6650 50  0001 C CNN
 F 3 "" H 5400 6650 50  0001 C CNN
-F 4 "C25501" H 5400 6650 50  0001 C CNN "LCSC Part"
+F 4 "C25725" H 5400 6650 50  0001 C CNN "LCSC Part"
 F 5 "Any manufacturer's part is acceptable." H 5400 6650 50  0001 C CNN "Notes"
-F 6 "Uniroyal 4D02WGJ0330TCE" H 5400 6650 50  0001 C CNN "Mfg. Part Numbers"
+F 6 "Uniroyal 4D02WGJ0103TCE" H 5400 6650 50  0001 C CNN "Mfg. Part Numbers"
 	1    5400 6650
 	0    -1   -1   0
@@
 	5600 6650 5600 6750
 Connection ~ 5600 6650
+$Comp
+L Device:R_Small R1
+U 1 1 61FFED1D
+P 7650 2900
+F 0 "R1" H 7591 2946 50  0000 R CNN
+F 1 "2k2" H 7591 2855 50  0000 R CNN
+F 2 "stdpads:R_0603" H 7650 2900 50  0001 C CNN
+F 3 "" H 7650 2900 50  0001 C CNN
+F 4 "C4190" H 7650 2900 50  0001 C CNN "LCSC Part"
+F 5 "Any manufacturer's part is acceptable." H 7650 2900 50  0001 C CNN "Notes"
+F 6 "Uniroyal 0603WAF2201T5E" H 7650 2900 50  0001 C CNN "Mfg. Part Numbers"
+	1    7650 2900
+	-1   0    0    -1
+$EndComp
+Text Label 7550 3200 0    50   ~ 0
+DONE
+$Comp
+L power:GND #PWR0159
+U 1 1 620004FF
+P 8050 2900
+F 0 "#PWR0159" H 8050 2650 50  0001 C CNN
+F 1 "GND" H 8050 2750 50  0000 C CNN
+F 2 "" H 8050 2900 50  0001 C CNN
+F 3 "" H 8050 2900 50  0001 C CNN
+	1    8050 2900
+	-1   0    0    -1
+$EndComp
+Wire Wire Line
+	7650 3000 7900 3000
+Wire Wire Line
+	7900 3000 7900 2900
+Wire Wire Line
+	7900 2900 8050 2900
+Wire Wire Line
+	7650 2800 7250 2800
 $EndSCHEMATC

Commit message: Generated gerbers and documenation PDFs
Parts:
- removed RN1, RN2, RN3, RN4, RN5: 4x33, stdpads:R4_0402, symbol Device:R_Pack04
- removed RN7: 4x10k, stdpads:R4_0402, symbol Device:R_Pack04
- added C30: 15p, stdpads:C_0603, symbol Device:C_Small
- added D1: White, stdpads:LED_0805, symbol Device:LED_Small_ALT
- added R10, R7, R8, R9: 10k, stdpads:R_0603, symbol Device:R_Small
- added R11, R2, R5: 47, stdpads:R_0603, symbol Device:R_Small
- added R6: 180, stdpads:R_0805, symbol Device:R_Small
- J1: value Memory Expansion -> IIgs RAM Exp.
- R1: value 2k2 -> 10k; LCSC Part C4190 -> C25804; Mfg. Part Numbers Uniroyal 0603WAF2201T5E -> Uniroyal 0603WAF1002T5E
- R3: value 100 -> 47; footprint stdpads:R_0805 -> stdpads:R_0603; LCSC Part C17408 -> C23182; Mfg. Part Numbers Uniroyal 0805W8F1000T5E -> Uniroyal 0603WAF470JT5E
- U1: value LCMXO2-640HC-4TG100C -> LCMXO2-TG100; Mfg. Part Numbers Lattice LCMXO2-640HC-4TG100C, Lattice LCMXO2-640HC-5TG100C, Lattice LCMXO2-640HC-6TG100C -> Lattice LCMXO2-640HC-4TG100C, Lattice LCMXO2-640HC-5TG100C, Lattice LCMXO2-640HC-6TG100C, Lattice LCMXO2-640HC-4TG100I, Lattice LCMXO2-640HC-5TG100I, Lattice LCMXO2-640HC-6TG100I, Lattice LCMXO2-1200HC-4TG100C, Lattice LCMXO2-1200HC-5TG100C, Lattice LCMXO2-1200HC-6TG100C, Lattice LCMXO2-1200HC-4TG100I, Lattice LCMXO2-1200HC-5TG100I, Lattice LCMXO2-1200HC-6TG100I
- U10, U9: Notes (none) -> Most 74LVC1G04 or 74AHC1G04 in SOT-353 package is acceptabl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
- U11: Notes (none) -> Most 1.2V regulator in SOT-23-5 package is acceptable.
- U2: Notes Most 166 MHz 128/256 Mbit SDRAM is acceptable. -> Most 166 MHz 128/256 Mbit x16 SDRAM is acceptable.
- U4: Notes (none) -> Most 74AHCT245 in TSSOP-20 package is acceptable.
- U5, U6, U7: Notes (none) -> Most 74LVC245 or 74AHC245 in TSSOP-20 package is acceptable.
Connections:
- net RD0r is gone; now on net RD0: U1.36 (PB10A)
- net RD1r is gone; now on net RD1: U1.37 (PB10B)
- net RD2r is gone; now on net RD3: U1.39 (PB10D/PCLKC2_1)
- net RD3r is gone; now on net RD2: U1.38 (PB10C/PCLKT2_1)
- net RD4r is gone; now on net RD5: U1.41 (PB12B)
- net RD5r is gone; now on net RD4: U1.40 (PB12A)
- net RD6r is gone; now on net RD6: U1.42 (PB12C)
- net RD7r is gone; now on net RD7: U1.43 (PB12D)
- net +3V3: now also R6.2, R7.1, R8.1, R9.1
- net AClk: now also R3.2
- net Ain3: now also U7.14 (B4)
- net Ain4: now also U7.15 (B3)
- net Ain5: now also U7.16 (B2)
- net Ain6: now also U7.13 (B5)
- net Ain7: now also U7.17 (B1)
- net Ain8: now also U7.12 (B6)
- net Ain9: now also U7.11 (B7)
- net DONE: now also R8.2
- net GND: now also C30.2, R10.1
- net RClk: now also R2.2
- net TCK: now also C30.1, R10.2, R11.1; no longer J2.1 (Pin_1)
- net ~CRAS~in: now also R5.1
- net ~INIT~: now also R9.2
- net ~PROG~: now also R7.2
- net at U4.19 (~OE~): now also U9.4 (Y); no longer R3.2
- net at U7.18 (B0): now also R5.2
- net at U10.4 (Y): now also R3.1, R2.1
- net LED: now reaches U1.34 (PB6C/PCLKT2_0)
- net LED: now also D1.1 (K)
- new net: D1.2 (A), R6.1
- new net TCKr: J2.1 (Pin_1), R11.2
- no-connect marks 21 -> 17
