File: Hardware/LCMXO2/RAM2GS.kicad_pcb (KiCad board)
At the start: 4 copper layers, 67.3 x 48.5 mm, 61 parts, among them J1 Memory Expansion, J2 JTAG, U1 LCMXO256-TQFP-100, U10 74LVC1G04GW, U11 SPIFlash-SON-8-1EP, U12 AP2127K-1.2, U2 W9812G6KH-6, U3 60M, U4 74AHCT245PW, U5 74LVC245APW, U6 74LVC245APW, U7 74LVC245APW, U8 AZ1117CH-3.3, U9 74LVC1G04GW

Commit message: finished MAX, LCMXO, iCE40?
Parts:
- removed the U11 at (53.5, 127.0)
- U11: renamed from U12; value AP2127K-1.2 -> AP2127K-1.2TRG1
- U8: value AZ1117CH-3.3 -> AZ1117CH-3.3TRG1
- moved FID4 6.14 mm to (48.5, 124.0)
Routing:
- net /MOSI: track 84.4 -> 0.00 mm, vias 2 -> 0
- net /S~CS~: track 82.5 -> 0.00 mm, vias 2 -> 0
- net /MISO: track 81.3 -> 0.00 mm, vias 2 -> 0
- net /SCK: track 80.1 -> 0.00 mm, vias 2 -> 0
- net GND: track 179.4 -> 175.3 mm, vias 222 -> 217
- net +3V3: track 266.0 -> 263.4 mm, vias 103 -> 100
- net +5V: track 198.4 -> 196.5 mm
- net /D3: track 1.75 -> 0.00 mm, vias 1 -> 0
- net /D2: track 1.75 -> 0.00 mm, vias 1 -> 0
- net /FD0: track 37.5 -> 36.7 mm
- added copper zone on F.Cu, net +1V2

Commit message: almost done
Parts:
- removed R1, R2: 22k, stdpads:R_0805
- added RN7: 4x10k, stdpads:R4_0402, F.Cu at (98.0, 103.7)
- U1: value LCMXO256-TQFP-100 -> LCMXO2-640HC-4TG100C
- moved C12 21.1 mm to (87.7, 118.2)
- moved C29 20.8 mm to (75.7, 104.8), turned to 270 degrees
- moved C11 17.3 mm to (90.7, 98.8), turned to 180 degrees
- moved C15 11.9 mm to (78.7, 98.8), turned to 180 degrees
- moved C14 7.99 mm to (92.2, 118.2), turned to 0 degrees
- moved C16 5.00 mm to (95.1, 112.3), turned to 90 degrees
- moved C13 4.50 mm to (81.9, 98.8), turned to 0 degrees
- moved C9 3.25 mm to (81.2, 118.2), turned to 180 degrees
- turned U1 to 90 degrees
Connections:
- U1 pad 1: /Dout0 -> /Din7
- U1 pad 10: +3V3 -> /CROWin0
- U1 pad 100: /RA7 -> +1V2
- U1 pad 11: Net-(U1-Pad11) -> (no net)
- U1 pad 12: GND -> /Ain1
- U1 pad 13: Net-(U1-Pad13) -> /Ain2
- U1 pad 14: /Din2 -> /Ain0
- U1 pad 15: /Din1 -> /~WE~in
- U1 pad 16: /Din3 -> /CROWin1
- U1 pad 17: /Din5 -> /~CRAS~in
- U1 pad 18: /Din4 -> /Ain7
- U1 pad 19: /Din7 -> /Ain5
- U1 pad 2: /Dout6 -> /Din6
- U1 pad 20: /Din6 -> /Ain4
- U1 pad 21: /Din0 -> /Ain3
- U1 pad 22: /~WE~in -> GND
- U1 pad 23: /Ain0 -> +3V3
- U1 pad 24: +3V3 -> /Ain6
- U1 pad 25: GND -> /Ain8
- U1 pad 26: /TMS -> +3V3
- U1 pad 27: /~CCAS~in -> Net-(U1-Pad27)
- U1 pad 28: /TCK -> Net-(U1-Pad28)
- U1 pad 29: /CROWin0 -> Net-(U1-Pad29)
- U1 pad 3: /Dout7 -> /Din0
- U1 pad 30: /CROWin1 -> Net-(U1-Pad30)
- U1 pad 31: /TDO -> Net-(U1-Pad31)
- U1 pad 32: Net-(U1-Pad32) -> /Ain9
- U1 pad 33: /TDI -> GND
- U1 pad 35: +1V2 -> Net-(U1-Pad35)
- U1 pad 36: Net-(U1-Pad36) -> /RD0r
- U1 pad 37: /Ain2 -> /RD1r
- U1 pad 38: /Ain1 -> /RD3r
- U1 pad 39: /PH2in -> /RD2r
- U1 pad 4: /Dout4 -> Net-(U1-Pad4)
- U1 pad 40: GND -> /RD5r
- U1 pad 41: +3V3 -> /RD4r
- U1 pad 42: GND -> /RD6r
- U1 pad 43: /~CRAS~in -> /RD7r
- U1 pad 44: /Ain7 -> GND
- U1 pad 45: /Ain5 -> Net-(U1-Pad45)
- U1 pad 46: /Ain4 -> +3V3
- U1 pad 47: /Ain3 -> Net-(U1-Pad47)
- U1 pad 48: Net-(U1-Pad48) -> /DQML
- U1 pad 49: /Ain6 -> /R~WE~
- U1 pad 5: /Dout5 -> +3V3
- U1 pad 50: /Ain8 -> +1V2
- U1 pad 51: /Ain9 -> /DQMH
- U1 pad 52: Net-(U1-Pad52) -> /R~CAS~
- U1 pad 53: /S~CS~ -> /CKE
- U1 pad 54: Net-(U1-Pad54) -> /R~RAS~
- U1 pad 55: /MISO -> +3V3
- U1 pad 56: /MOSI -> GND
- U1 pad 57: Net-(U1-Pad57) -> /R~CS~
- U1 pad 58: /SCK -> /BA0
- U1 pad 59: Net-(U1-Pad59) -> /RA11
- U1 pad 6: /Dout3 -> GND
- U1 pad 60: +3V3 -> /BA1
- U1 pad 61: Net-(U1-Pad61) -> (no net)
- U1 pad 62: GND -> /AClk
- U1 pad 63: Net-(U1-Pad63) -> /RA9
- U1 pad 64: /RD0r -> /RA10
- U1 pad 65: /RD1r -> /RA8
- U1 pad 66: /RD3r -> /RA0
- U1 pad 67: /RD2r -> /RA1
- U1 pad 68: /RD5r -> /RA6
- U1 pad 69: /RD4r -> /RA2
- U1 pad 7: /Dout1 -> Net-(U1-Pad7)
- U1 pad 70: /RD6r -> /RA5
- U1 pad 71: /RD7r -> /RA3
- U1 pad 72: /DQML -> GND
- U1 pad 73: /R~RAS~ -> +3V3
- U1 pad 74: +3V3 -> /RA4
- U1 pad 75: GND -> /RA7
- U1 pad 76: /R~WE~ -> /DONE
- U1 pad 77: /R~CS~ -> /~INIT~
- U1 pad 78: /DQMH -> /Dout6
- U1 pad 79: /BA0 -> GND
- U1 pad 8: /Dout2 -> /PH2in
- U1 pad 80: /R~CAS~ -> +3V3
- U1 pad 81: /RA11 -> /~PROG~
- U1 pad 82: /CKE -> /Dout7
- U1 pad 83: /BA1 -> /Dout4
- U1 pad 84: GND -> /Dout5
- U1 pad 85: /RA9 -> /Dout3
- U1 pad 86: /AClk -> /Dout1
- U1 pad 87: /RA10 -> /Dout2
- U1 pad 88: +3V3 -> /Din2
- U1 pad 89: /RA1 -> (no net)
- U1 pad 9: Net-(U1-Pad9) -> /~CCAS~in
- U1 pad 90: +1V2 -> /TMS
- U1 pad 91: /RA6 -> /TCK
- U1 pad 92: +3V3 -> GND
- U1 pad 93: GND -> +3V3
- U1 pad 94: /RA2 -> /TDI
- U1 pad 95: /RA5 -> /TDO
- U1 pad 96: /RA8 -> /Din1
- U1 pad 97: /RA3 -> /Din3
- U1 pad 98: /RA0 -> /Din5
- U1 pad 99: /RA4 -> /Din4
- U4 pad 18: /Dout0 -> /DONE
Routing:
- net /DONE: track 0.00 -> 59.7 mm, vias 0 -> 2
- net /~PROG~: track 0.00 -> 45.1 mm, vias 0 -> 2
- net /~INIT~: track 0.00 -> 41.7 mm, vias 0 -> 2
- net +1V2: track 105.8 -> 86.7 mm, vias 9 -> 6
- net /Dout6: track 7.88 -> 19.6 mm, vias 0 -> 2
- net /Ain9: track 30.1 -> 41.8 mm, vias 0 -> 2
- net /~WE~in: track 9.59 -> 20.4 mm, vias 0 -> 2
- net /Ain0: track 9.81 -> 19.5 mm, vias 0 -> 2
- net /CROWin0: track 11.9 -> 21.1 mm, vias 0 -> 2
- net /TCK: track 30.5 -> 39.3 mm
- net /Dout0: track 7.94 -> 0.00 mm
- net /Din0: track 6.85 -> 14.3 mm
- net /Din6: track 6.62 -> 14.0 mm
- net /~CCAS~in: track 10.9 -> 18.2 mm, vias 0 -> 2
- net /Din7: track 6.52 -> 13.6 mm
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
Commit message: more
Parts:
- added R1: 2k2, stdpads:R_0603, F.Cu at (78.0, 119.0)
Routing:
- net /DONE: track 59.7 -> 61.5 mm
- net GND: track 177.6 -> 179.2 mm
Changed lines of the file:
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@@
     (thickness 1.6)
     (drawings 47)
-    (tracks 2247)
+    (tracks 2255)
     (zones 0)
-    (modules 59)
+    (modules 60)
     (nets 148)
   )
@@
     (mod_text_size 1 1)
     (mod_text_width 0.15)
-    (pad_size 1.475 0.3)
+    (pad_size 0.7 0.95)
     (pad_drill 0)
     (pad_to_mask_clearance 0.075)
@@
     (add_net "Net-(U9-Pad1)")
   )
+  (module stdpads:R_0603 (layer F.Cu)
+    (at 77.95 119 90)
+    (tags resistor)
+    (solder_mask_margin 0.05)
+    (solder_paste_margin -0.05)
+    (attr smd)
+    (fp_text reference R1 (at 0 0 90) (layer F.Fab)
+      (effects (font (size 0.254 0.254) (thickness 0.0635)))
+    )
+    (fp_text value 2k2 (at 0 0.25 90) (layer F.Fab)
+      (effects (font (size 0.127 0.127) (thickness 0.03175)))
+    )
+    (fp_line (start -0.8 0.4) (end -0.8 -0.4) (layer F.Fab) (width 0.1))
+    (fp_line (start -0.8 -0.4) (end 0.8 -0.4) (layer F.Fab) (width 0.1))
+    (fp_line (start 0.8 -0.4) (end 0.8 0.4) (layer F.Fab) (width 0.1))
+    (fp_line (start 0.8 0.4) (end -0.8 0.4) (layer F.Fab) (width 0.1))
+    (fp_line (start -0.162779 -0.51) (end 0.162779 -0.51) (layer F.SilkS) (width 0.12))
+    (fp_line (start -0.162779 0.51) (end 0.162779 0.51) (layer F.SilkS) (width 0.12))
+    (fp_line (start -1.4 0.7) (end -1.4 -0.7) (layer F.CrtYd) (width 0.05))
+    (fp_line (start -1.4 -0.7) (end 1.4 -0.7) (layer F.CrtYd) (width 0.05))
+    (fp_line (start 1.4 -0.7) (end 1.4 0.7) (layer F.CrtYd) (width 0.05))
+    (fp_line (start 1.4 0.7) (end -1.4 0.7) (layer F.CrtYd) (width 0.05))
+    (fp_text user %R (at 0 0 90) (layer F.SilkS) hide
+      (effects (font (size 0.254 0.254) (thickness 0.0635)))
+    )
+    (pad 1 smd roundrect (at -0.8 0 90) (size 0.7 0.95) (layers F.Cu F.Paste F.Mask) (roundrect_rratio 0.25)
+      (net 42 /Dout7))
+    (pad 2 smd roundrect (at 0.8 0 90) (size 0.7 0.95) (layers F.Cu F.Paste F.Mask) (roundrect_rratio 0.25)
+      (net 1 GND))
+    (model ${KISYS3DMOD}/Resistor_SMD.3dshapes/R_0603_1608Metric.wrl
+      (at (xyz 0 0 0))
+      (scale (xyz 1 1 1))
+      (rotate (xyz 0 0 0))
+    )
+  )
   (module stdpads:TQFP-100_14x14mm_P0.5mm (layer F.Cu)
     (at 85.4 108.55 90)
@@
   (via (at 84.9 117.8) (size 0.5) (drill 0.2) (layers F.Cu B.Cu) (net 1))
   (via (at 85.1 121.05) (size 0.5) (drill 0.2) (layers F.Cu B.Cu) (net 1))
-  (via (at 76.8 120.65) (size 0.5) (drill 0.2) (layers F.Cu B.Cu) (net 1))
   (via (at 90.5 119.1) (size 0.5) (drill 0.2) (layers F.Cu B.Cu) (net 1))
   (via (at 82.4 97.95) (size 0.5) (drill 0.2) (layers F.Cu B.Cu) (net 1))
@@
   (via (at 83.2 105.8) (size 0.5) (drill 0.2) (layers F.Cu B.Cu) (net 1))
   (via (at 86.15 106.8) (size 0.5) (drill 0.2) (layers F.Cu B.Cu) (net 1))
+  (via (at 76.35 119.7) (size 0.5) (drill 0.2) (layers F.Cu B.Cu) (net 1))
+  (segment (start 79.55 118.2) (end 79.6 118.25) (width 0.15) (layer F.Cu) (net 1))
+  (segment (start 77.95 118.2) (end 79.55 118.2) (width 0.15) (layer F.Cu) (net 1))
   (segment (start 88.138 135.382) (end 88.138 130.048) (width 0.15) (layer F.Cu) (net 8))
   (via (at 88.138 130.048) (size 0.5) (drill 0.2) (layers F.Cu B.Cu) (net 8))
@@
   (segment (start 82.9 117.1) (end 83.1 117.3) (width 0.15) (layer F.Cu) (net 41))
   (segment (start 82.9 116.2125) (end 82.9 117.1) (width 0.15) (layer F.Cu) (net 41))
+  (segment (start 77.95 120.35) (end 76.7 121.6) (width 0.15) (layer F.Cu) (net 42))
   (segment (start 76.7 121.6) (end 76.7 122.5) (width 0.15) (layer F.Cu) (net 42))
-  (segment (start 78.95 119.35) (end 76.7 121.6) (width 0.15) (layer F.Cu) (net 42))
-  (segment (start 82.1 119.35) (end 78.95 119.35) (width 0.15) (layer F.Cu) (net 42))
-  (segment (start 82.8 118.65) (end 82.1 119.35) (width 0.15) (layer F.Cu) (net 42))
+  (segment (start 77.95 119.8) (end 77.95 120.35) (width 0.15) (layer F.Cu) (net 42))
+  (segment (start 82.1 119.35) (end 79.15 119.35) (width 0.15) (layer F.Cu) (net 42))
+  (segment (start 79.15 119.35) (end 78.7 119.8) (width 0.15) (layer F.Cu) (net 42))
+  (segment (start 78.7 119.8) (end 77.95 119.8) (width 0.15) (layer F.Cu) (net 42))
   (segment (start 82.8 117.5) (end 82.8 118.65) (width 0.15) (layer F.Cu) (net 42))
+  (segment (start 82.8 118.65) (end 82.1 119.35) (width 0.15) (layer F.Cu) (net 42))
   (segment (start 82.4 117.1) (end 82.8 117.5) (width 0.15) (layer F.Cu) (net 42))
   (segment (start 82.4 116.2125) (end 82.4 117.1) (width 0.15) (layer F.Cu) (net 42))
@@
   (via (at 99.75 102.4) (size 0.5) (drill 0.2) (layers F.Cu B.Cu) (net 146))
   (via (at 79.4 117.35) (size 0.5) (drill 0.2) (layers F.Cu B.Cu) (net 146))
-  (segment (start 75.4 121.35) (end 75.4 122.5) (width 0.15) (layer F.Cu) (net 146))
-  (segment (start 79.4 117.35) (end 75.4 121.35) (width 0.15) (layer F.Cu) (net 146))
   (segment (start 79.4 116.2125) (end 79.4 117.35) (width 0.15) (layer F.Cu) (net 146))
   (segment (start 102.1 98.75) (end 96.85 93.5) (width 0.15) (layer B.Cu) (net 146))
@@
   (segment (start 87.45 101.4) (end 87.45 102.9) (width 0.15) (layer B.Cu) (net 146))
   (segment (start 99.75 102.4) (end 100.1 102.75) (width 0.15) (layer B.Cu) (net 146))
+  (segment (start 75.4 121.35) (end 75.4 122.5) (width 0.15) (layer F.Cu) (net 146))
+  (segment (start 76.85 119.9) (end 75.4 121.35) (width 0.15) (layer F.Cu) (net 146))
+  (segment (start 76.85 117.65) (end 76.85 119.9) (width 0.15) (layer F.Cu) (net 146))
+  (segment (start 78.2875 116.2125) (end 76.85 117.65) (width 0.15) (layer F.Cu) (net 146))
+  (segment (start 79.4 116.2125) (end 78.2875 116.2125) (width 0.15) (layer F.Cu) (net 146))
   (segment (start 98.75 102.6) (end 98.746447 102.6) (width 0.15) (layer F.Cu) (net 147))
   (segment (start 98.746447 102.6) (end 98.226777 103.11967) (width 0.15) (layer F.Cu) (net 147))
@@
     (connect_pads (clearance 0.15))
     (min_thickness 0.15)
-    (fill yes (arc_segments 32) (thermal_gap 0.15) (thermal_bridge_width 0.3))
+    (fill (arc_segments 32) (thermal_gap 0.15) (thermal_bridge_width 0.3))
     (polygon
       (pts
@@
     (connect_pads (clearance 0.15))
     (min_thickness 0.15)
-    (fill yes (arc_segments 32) (thermal_gap 0.15) (thermal_bridge_width 0.3))
+    (fill (arc_segments 32) (thermal_gap 0.15) (thermal_bridge_width 0.3))
     (polygon
       (pts
@@
     (connect_pads (clearance 0.15))
     (min_thickness 0.15)
-    (fill yes (arc_segments 32) (thermal_gap 0.15) (thermal_bridge_width 0.3))
+    (fill (arc_segments 32) (thermal_gap 0.15) (thermal_bridge_width 0.3))
     (polygon
       (pts
@@
     (connect_pads (clearance 0.15))
     (min_thickness 0.15)
-    (fill yes (arc_segments 32) (thermal_gap 0.15) (thermal_bridge_width 0.3))
+    (fill (arc_segments 32) (thermal_gap 0.15) (thermal_bridge_width 0.3))
     (polygon
       (pts
@@
     (connect_pads (clearance 0.1524))
     (min_thickness 0.1524)
-    (fill yes (arc_segments 32) (thermal_gap 0.1524) (thermal_bridge_width 0.3))
+    (fill (arc_segments 32) (thermal_gap 0.1524) (thermal_bridge_width 0.3))
     (polygon
       (pts

Commit message: Generated gerbers and documenation PDFs
Parts:
- removed RN1, RN2, RN3, RN4, RN5: 4x33, stdpads:R4_0402
- removed RN7: 4x10k, stdpads:R4_0402
- added C30: 15p, stdpads:C_0603, F.Cu at (98.0, 104.0)
- added D1: White, stdpads:LED_0805, F.Cu at (71.3, 102.7)
- added R10: 10k, stdpads:R_0603, F.Cu at (97.0, 103.0)
- added R11: 47, stdpads:R_0603, F.Cu at (97.8, 98.2)
- added R2: 47, stdpads:R_0603, F.Cu at (70.5, 108.0)
- added R5: 47, stdpads:R_0603, F.Cu at (96.8, 115.8)
- added R6: 180, stdpads:R_0805, F.Cu at (71.3, 104.6)
- added R7: 10k, stdpads:R_0603, F.Cu at (99.1, 105.0)
- added R8: 10k, stdpads:R_0603, F.Cu at (75.6, 119.7)
- added R9: 10k, stdpads:R_0603, F.Cu at (72.8, 119.7)
- J1: value Memory Expansion -> IIgs RAM Exp.
- R1: value 2k2 -> 10k
- R3: value 100 -> 47; footprint stdpads:R_0805 -> stdpads:R_0603
- U1: value LCMXO2-640HC-4TG100C -> LCMXO2-TG100
- moved R3 17.8 mm to (73.2, 108.0)
Connections:
- J2 pad 1: /TCK -> /TCKr
- R3 pad 1: Net-(R3-Pad1) -> Net-(R2-Pad1)
- R3 pad 2: Net-(R3-Pad2) -> /AClk
- U1 pad 34: Net-(U1-Pad34) -> /LED
- U1 pad 36: /RD0r -> /RD0
- U1 pad 37: /RD1r -> /RD1
- U1 pad 38: /RD3r -> /RD2
- U1 pad 39: /RD2r -> /RD3
- U1 pad 40: /RD5r -> /RD4
- U1 pad 41: /RD4r -> /RD5
- U1 pad 42: /RD6r -> /RD6
- U1 pad 43: /RD7r -> /RD7
- U10 pad 4: Net-(RN1-Pad1) -> Net-(R2-Pad1)
- U4 pad 19: Net-(R3-Pad2) -> Net-(U4-Pad19)
- U7 pad 11: Net-(RN5-Pad4) -> /Ain9
- U7 pad 12: Net-(RN5-Pad3) -> /Ain8
- U7 pad 13: Net-(RN5-Pad2) -> /Ain6
- U7 pad 14: Net-(RN5-Pad1) -> /Ain3
- U7 pad 15: Net-(RN4-Pad4) -> /Ain4
- U7 pad 16: Net-(RN4-Pad3) -> /Ain5
- U7 pad 17: Net-(RN4-Pad2) -> /Ain7
- U9 pad 4: Net-(R3-Pad1) -> Net-(U4-Pad19)
Routing:
- net /DONE: track 61.5 -> 8.60 mm, vias 2 -> 0
- net /RD1r: track 26.8 -> 0.00 mm, vias 2 -> 0
- net /RD4r: track 26.2 -> 0.00 mm, vias 2 -> 0
- net /RD2r: track 25.8 -> 0.00 mm, vias 2 -> 0
- net /RD0r: track 25.4 -> 0.00 mm, vias 2 -> 0
- net /RD7r: track 24.9 -> 0.00 mm, vias 2 -> 0
- net /RD1: track 19.3 -> 44.0 mm
- net /RD5r: track 24.7 -> 0.00 mm, vias 2 -> 0
- net /RD3r: track 24.7 -> 0.00 mm, vias 2 -> 0
- net /RD3: track 19.5 -> 43.5 mm
- net /RD6r: track 23.7 -> 0.00 mm, vias 2 -> 0
- net /RD0: track 18.6 -> 42.2 mm
- net /RD2: track 19.4 -> 42.0 mm
- net /RD5: track 20.3 -> 42.1 mm
- net /RD4: track 20.0 -> 41.4 mm
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- added copper zone on F.Cu, net +3V3
Other:
- board text added: "D20C"

Commit message: Updated LCMXO2 board, fixed GND via
Routing:
- net GND: vias 211 -> 212
- net (no net): vias 1 -> 0
Changed lines of the file:
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@@
     (add_net "Net-(U9-Pad1)")
+  )
+  (module stdpads:R_0603 (layer F.Cu)
+    (at 75.6 119.65)
+    (tags resistor)
+    (solder_mask_margin 0.05)
+    (solder_paste_margin -0.05)
+    (attr smd)
+    (fp_text reference R8 (at 0 0) (layer F.Fab)
+      (effects (font (size 0.254 0.254) (thickness 0.0635)))
+    )
+    (fp_text value 10k (at 0 0.25) (layer F.Fab)
+      (effects (font (size 0.127 0.127) (thickness 0.03175)))
+    )
+    (fp_line (start -0.8 0.4) (end -0.8 -0.4) (layer F.Fab) (width 0.1))
+    (fp_line (start -0.8 -0.4) (end 0.8 -0.4) (layer F.Fab) (width 0.1))
+    (fp_line (start 0.8 -0.4) (end 0.8 0.4) (layer F.Fab) (width 0.1))
+    (fp_line (start 0.8 0.4) (end -0.8 0.4) (layer F.Fab) (width 0.1))
+    (fp_line (start -0.162779 -0.51) (end 0.162779 -0.51) (layer F.SilkS) (width 0.12))
+    (fp_line (start -0.162779 0.51) (end 0.162779 0.51) (layer F.SilkS) (width 0.12))
+    (fp_line (start -1.4 0.7) (end -1.4 -0.7) (layer F.CrtYd) (width 0.05))
+    (fp_line (start -1.4 -0.7) (end 1.4 -0.7) (layer F.CrtYd) (width 0.05))
+    (fp_line (start 1.4 -0.7) (end 1.4 0.7) (layer F.CrtYd) (width 0.05))
+    (fp_line (start 1.4 0.7) (end -1.4 0.7) (layer F.CrtYd) (width 0.05))
+    (fp_text user %R (at 0 0) (layer F.SilkS) hide
+      (effects (font (size 0.254 0.254) (thickness 0.0635)))
+    )
+    (pad 1 smd roundrect (at -0.8 0) (size 0.7 0.95) (layers F.Cu F.Paste F.Mask) (roundrect_rratio 0.25)
+      (net 37 +3V3))
+    (pad 2 smd roundrect (at 0.8 0) (size 0.7 0.95) (layers F.Cu F.Paste F.Mask) (roundrect_rratio 0.25)
+      (net 122 /DONE))
+    (model ${KISYS3DMOD}/Resistor_SMD.3dshapes/R_0603_1608Metric.wrl
+      (at (xyz 0 0 0))
+      (scale (xyz 1 1 1))
+      (rotate (xyz 0 0 0))
+    )
   )
   (module stdpads:TSSOP-20_4.4x6.5mm_P0.65mm (layer F.Cu)
@@
       (rotate (xyz 0 0 0))
     )
-  )
-  (module stdpads:R_0603 (layer F.Cu)
-    (at 75.6 119.65)
-    (tags resistor)
-    (solder_mask_margin 0.05)
-    (solder_paste_margin -0.05)
-    (attr smd)
-    (fp_text reference R8 (at 0 0) (layer F.Fab)
-      (effects (font (size 0.254 0.254) (thickness 0.0635)))
-    )
-    (fp_text value 10k (at 0 0.25) (layer F.Fab)
-      (effects (font (size 0.127 0.127) (thickness 0.03175)))
-    )
-    (fp_line (start 1.4 0.7) (end -1.4 0.7) (layer F.CrtYd) (width 0.05))
-    (fp_line (start 1.4 -0.7) (end 1.4 0.7) (layer F.CrtYd) (width 0.05))
-    (fp_line (start -1.4 -0.7) (end 1.4 -0.7) (layer F.CrtYd) (width 0.05))
-    (fp_line (start -1.4 0.7) (end -1.4 -0.7) (layer F.CrtYd) (width 0.05))
-    (fp_line (start -0.162779 0.51) (end 0.162779 0.51) (layer F.SilkS) (width 0.12))
-    (fp_line (start -0.162779 -0.51) (end 0.162779 -0.51) (layer F.SilkS) (width 0.12))
-    (fp_line (start 0.8 0.4) (end -0.8 0.4) (layer F.Fab) (width 0.1))
-    (fp_line (start 0.8 -0.4) (end 0.8 0.4) (layer F.Fab) (width 0.1))
-    (fp_line (start -0.8 -0.4) (end 0.8 -0.4) (layer F.Fab) (width 0.1))
-    (fp_line (start -0.8 0.4) (end -0.8 -0.4) (layer F.Fab) (width 0.1))
-    (fp_text user %R (at 0 0) (layer F.SilkS) hide
-      (effects (font (size 0.254 0.254) (thickness 0.0635)))
-    )
-    (pad 2 smd roundrect (at 0.8 0) (size 0.7 0.95) (layers F.Cu F.Paste F.Mask) (roundrect_rratio 0.25)
-      (net 122 /DONE))
-    (pad 1 smd roundrect (at -0.8 0) (size 0.7 0.95) (layers F.Cu F.Paste F.Mask) (roundrect_rratio 0.25)
-      (net 37 +3V3))
   )
   (module stdpads:LED_0805 (layer F.Cu)
@@
     (pad 1 smd roundrect (at -0.75 0 270) (size 0.85 0.95) (layers F.Cu F.Paste F.Mask) (roundrect_rratio 0.25)
       (net 37 +3V3))
-    (model ${KISYS3DMOD}/Capacitor_SMD.3dshapes/C_0603_1608Metric.wrl
-      (at (xyz 0 0 0))
-      (scale (xyz 1 1 1))
-      (rotate (xyz 0 0 0))
-    )
   )
   (module stdpads:Fiducial (layer F.Cu)
@@
   (gr_line (start 55.372 139.192) (end 55.372 132.08) (layer Edge.Cuts) (width 0.15))
   (gr_line (start 112.776 139.7) (end 55.88 139.7) (layer Edge.Cuts) (width 0.15))
-  (via (at 107.15 118.5) (size 0.5) (drill 0.2) (layers F.Cu B.Cu) (net 0) (status 40000))
+  (via (at 107.15 118.5) (size 0.5) (drill 0.2) (layers F.Cu B.Cu) (net 1) (status 40000))
   (via (at 85.471 94.996) (size 0.5) (drill 0.2) (layers F.Cu B.Cu) (net 1))
   (via (at 80.391 94.742) (size 0.5) (drill 0.2) (layers F.Cu B.Cu) (net 1))

Commit message: Documentation update
Connections:
- U1 pad 62: /AClk -> /RA9
- U1 pad 63: /RA9 -> /AClk
Routing:
- net /RA9: track 18.7 -> 19.8 mm
