File: Hardware/LCMXO2/RAM2GS.kicad_pcb (KiCad board)
At the start: 4 copper layers, 67.3 x 48.5 mm, 64 parts, among them J1 IIgs RAM Exp., J2 JTAG, U1 LCMXO2-TG100, U10 74LVC1G04GW, U11 AP2127K-1.2TRG1, U2 W9812G6KH-6, U3 60M, U4 74AHCT245PW, U5 74LVC245APW, U6 74LVC245APW, U7 74LVC245APW, U8 AZ1117CH-3.3TRG1, U9 74LVC1G04GW

Commit message: 2.1?
Parts:
- added G***: LOGO, LOGO, F.Cu at (67.2, 95.2)
- added G***: LOGO, LOGO, F.Cu at (87.5, 95.0)
- added R12: 47, stdpads:R_0603, F.Cu at (73.2, 106.5)
- added R13: 47, stdpads:R_0603, F.Cu at (75.2, 110.5)
- D1: value White -> Amber
- R6: value 180 -> 220
- turned U10 to 90 degrees
- turned U11 to 0 degrees
- turned U2 to -90 degrees
- turned U9 to -90 degrees
- renumbered H5 to H3, H3 to H5
Connections:
- net /AClk renamed /FCLK
- net /RClk renamed /RCLK
- net /R~CAS~ renamed /R~{CAS}
- net /R~CS~ renamed /R~{CS}
- net /R~RAS~ renamed /R~{RAS}
- net /R~WE~ renamed /R~{WE}
- net /~CCAS~ renamed /~{CCAS}
- net /~CCAS~in renamed /~{CCAS}in
- net /~CRAS~ renamed /~{CRAS}
- net /~CRAS~in renamed /~{CRAS}in
- net /~CROMSEL~ renamed /~{CROMSEL}
- net /~CSEL~ renamed /~{CSEL}
- net /~FWE~ renamed /~{FWE}
- net /~INIT~ renamed /~{INIT}
- net /~PROG~ renamed /~{PROG}
- net /~WE~in renamed /~{WE}in
- net Net-(R2-Pad1) renamed /~{C60M}
- net Net-(U10-Pad2) renamed /C60M
- J2 pad 10: Net-(J2-Pad10) -> unconnected-(J2-Pin_10-Pad10)
- J2 pad 8: Net-(J2-Pad8) -> unconnected-(J2-Pin_8-Pad8)
- J2 pad 9: Net-(J2-Pad9) -> unconnected-(J2-Pin_9-Pad9)
- U1 pad 27: Net-(U1-Pad27) -> unconnected-(U1-PB4A/CSSPIN-Pad27)
- U1 pad 28: Net-(U1-Pad28) -> unconnected-(U1-PB4B-Pad28)
- U1 pad 29: Net-(U1-Pad29) -> unconnected-(U1-PB4C-Pad29)
- U1 pad 30: Net-(U1-Pad30) -> unconnected-(U1-PB4D-Pad30)
- U1 pad 31: Net-(U1-Pad31) -> unconnected-(U1-PB6A/MCLK/CCLK-Pad31)
- U1 pad 35: Net-(U1-Pad35) -> unconnected-(U1-PB6D/PCLKC_0-Pad35)
- U1 pad 4: Net-(U1-Pad4) -> unconnected-(U1-PL2D/PCLKC3_2-Pad4)
- U1 pad 45: Net-(U1-Pad45) -> unconnected-(U1-PB14A-Pad45)
- U1 pad 47: Net-(U1-Pad47) -> /BA1
- U1 pad 60: /BA1 -> /RCLKout
- U1 pad 7: Net-(U1-Pad7) -> unconnected-(U1-PL3A-Pad7)
- U10 pad 1: Net-(U10-Pad1) -> unconnected-(U10-NC-Pad1)
- U11 pad 4: Net-(U11-Pad4) -> unconnected-(U11-NC-Pad4)
- U9 pad 1: Net-(U9-Pad1) -> unconnected-(U9-NC-Pad1)
Routing:
- net /BA1: track 32.8 -> 37.5 mm
- net /RCLK: track 9.42 -> 13.5 mm
- net /LED: track 20.3 -> 24.3 mm, vias 0 -> 2
- net /RCLKout: track 0.00 -> 3.94 mm
- net /FCLK: track 3.94 -> 6.18 mm
- net GND: track 177.9 -> 179.2 mm, vias 212 -> 211
- net /C60M: track 4.18 -> 4.91 mm
- net +3V3: track 262.3 -> 261.7 mm, vias 104 -> 103
Other:
- net class Default removed
- rule pad_to_mask_clearance: 0.075 -> 0.0762
- rule solder_mask_min_width: 0.1 -> 0.127
- board text added: "D21C"
- board text added: "JLCJLCJLCJLC"
- board text removed: "4201D"
- board text removed: "8 MB RAM"
- board text removed: "D20C"
- board text removed: "GW"
- board text removed: "Garrett’s Workshop"
- board text removed: "for Apple IIgs"

Commit message: RC 2.2
Parts:
- J2: footprint Connector:Tag-Connect_TC2050-IDC-FP_2x05_P1.27mm_Vertical -> stdpads:Tag-Connect_TC2050-IDC-FP_2x05_P1.27mm_Vertical
- R8, R9: value 10k -> DNP
- U1: value LCMXO2-TG100 -> LCMXO2-640HC-TG100C
Connections:
- J1 pad 11: +5V -> 5VC
Routing:
- net /TDO: track 33.5 -> 32.4 mm
- net GND: track 179.2 -> 178.2 mm
Other:
- board text added: "D22C"
- board text removed: "D21C"

Commit message: RC
Parts:
- C30: value 15p -> 22p
- U1: value LCMXO2-640HC-TG100C -> LCMXO2-640HC-4TG100C
Connections:
- R1 pad 2: GND -> +3V3
Routing:
- net +5V: track 196.5 -> 193.1 mm
- net +3V3: track 261.8 -> 262.3 mm, vias 103 -> 105
