File: Hardware/LCMXO2/RAM2GS.kicad_pcb (KiCad board)
At the start: 4 copper layers, 67.3 x 48.5 mm, 68 parts, among them J1 IIgs RAM Exp., J2 JTAG, U1 LCMXO2-640HC-4TG100C, U10 74LVC1G04GW, U11 AP2127K-1.2TRG1, U2 W9812G6KH-6, U3 60M, U4 74AHCT245PW, U5 74LVC245APW, U6 74LVC245APW, U7 74LVC245APW, U8 AZ1117CH-3.3TRG1, U9 74LVC1G04GW

Commit message: 2.2
Parts:
- H1, H2, H3, H4, H5: value (none) -> ~
- R2, R3: value 47 -> DNP
- U10: value 74LVC1G04GW -> DNP

Commit message: RC D.2.3
Connections:
- U1 pad 11: (no net) -> +3V3
- U1 pad 61: (no net) -> unconnected-(U1-NC-Pad61)
- U1 pad 89: (no net) -> unconnected-(U1-NC-Pad89)
- U2 pad 40: (no net) -> unconnected-(U2-NC-Pad40)
Routing:
- net +3V3: track 262.3 -> 264.6 mm, vias 105 -> 107
Other:
- board text added: "D23C"
- board text removed: "D22C"
