File: Hardware/LCMXO2/RAM2GS.kicad_sch (KiCad schematic)
At the start: 66 parts, among them J1 IIgs RAM Exp., J2 JTAG, U1 LCMXO2-TG100, U10 74LVC1G04GW, U11 AP2127K-1.2TRG1, U2 W9812G6KH-6, U3 60M, U4 74AHCT245PW, U5 74LVC245APW, U6 74LVC245APW, U7 74LVC245APW, U8 AZ1117CH-3.3TRG1, U9 74LVC1G04GW

Commit message: RC 2.2
Parts:
- C1, C2, C26, C3, C4: Mfg. Part Numbers Samsung CL21A106KAYNNNE -> (none); Notes 10V or higher. Any manufacturer's part is acceptable but Sa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 -> (none)
- C10, C11, C12, C13, C14, C15, C16, C17, C18, C19, C20, C21, C22, C23, C24, C25, C27, C28, C29, C5, C6, C7, C8, C9: Mfg. Part Numbers Samsung CL10A225KO8NNNC -> (none); Notes 10V or higher. Any manufacturer's part is acceptable but Sa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 -> (none)
- C30: LCSC Part C1644 -> C1653; Mfg. Part Numbers Samsung CL10C150JB8NNNC -> (none); Notes 10V or higher. Any manufacturer's part is acceptable but Sa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 -> (none)
- D1: LCSC Part (none) -> C284932; Notes Any manufacturer's part is acceptable. -> (none)
- FID1, FID2, FID3, FID4: Notes DNP - SMT vision system fiducial -> (none)
- H1, H2, H4, H5: Notes DNP - mounting hole for solder paste printing -> (none)
- H3: Notes DNP - mounting hole -> (none)
- J1: Notes DNP - edge connector -> (none)
- J2: footprint Connector:Tag-Connect_TC2050-IDC-FP_2x05_P1.27mm_Vertical -> stdpads:Tag-Connect_TC2050-IDC-FP_2x05_P1.27mm_Vertical; Notes DNP - test pad connector -> (none)
- R1, R10, R7: Mfg. Part Numbers Uniroyal 0603WAF1002T5E -> (none); Notes Any manufacturer's part is acceptable. -> (none)
- R11, R12, R13, R2, R3, R5: Mfg. Part Numbers Uniroyal 0603WAF470JT5E -> (none); Notes Any manufacturer's part is acceptable. -> (none)
- R4: Mfg. Part Numbers Uniroyal 0805W8F0000T5E -> (none); Notes Any manufacturer's part is acceptable. -> (none)
- R6: Mfg. Part Numbers Uniroyal 0805W8F2200T5E -> (none); Notes Any manufacturer's part is acceptable. -> (none)
- R8, R9: value 10k -> DNP; LCSC Part C25804 -> (none); Mfg. Part Numbers Uniroyal 0603WAF1002T5E -> (none); Notes Any manufacturer's part is acceptable. -> (none)
- U1: value LCMXO2-TG100 -> LCMXO2-640HC-TG100C; Mfg. Part Numbers Lattice LCMXO2-640HC-4TG100C, Lattice LCMXO2-640HC-5TG100C,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 -> (none)
- U10, U9: Mfg. Part Numbers NXP 74LVC1G04GW, TI SN74LVC1G04DCK -> (none); Notes Most 74LVC1G04 or 74AHC1G04 in SOT-353 package is acceptabl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 -> (none)
- U11: Mfg. Part Numbers Diodes AP2127K-1.2TRG1, Torex XC6228D122VR -> (none); Notes Most 1.2V regulator in SOT-23-5 package is acceptable. -> (none)
- U2: Mfg. Part Numbers Winbond W9812G6KH-6, Winbond W9812G6KH-6I, Winbond W9825G6K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 -> (none); Notes Most 166 MHz 128/256 Mbit x16 SDRAM is acceptable. -> (none)
- U3: Mfg. Part Numbers SiTime SIT1602AI-82-33E-60.000000Y, Shenzhen SCTF S7D60.000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 -> (none); Notes Most 60-62.5 MHz 3.3V crystal oscillator or silicon oscilla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 -> (none)
- U4: Mfg. Part Numbers NXP 74AHCT245PW, TI SN74AHCT245PW -> (none); Notes Most 74AHCT245 in TSSOP-20 package is acceptable. -> (none)
- U5, U6, U7: Mfg. Part Numbers NXP 74LVC245APW, TI SN74LVC245APW -> (none); Notes Most 74LVC245 or 74AHC245 in TSSOP-20 package is acceptable. -> (none)
- U8: Mfg. Part Numbers Diodes AZ1117CH-3.3TRG1, Diodes AZ1117EH-3.3TRG1 -> (none); Notes Most 1117-type 3.3V regulator in SOT-223 package is accepta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 -> (none)
Connections:
- net +5V: no longer J1.11 (Pin_11)
- new net 5VC: J1.11 (Pin_11)

Commit message: RC
Parts:
- C30: value 15p -> 22p
- U1: value LCMXO2-640HC-TG100C -> LCMXO2-640HC-4TG100C
Connections:
- net +3V3: now also R1.2
- net GND: no longer R1.2
Other:
- moved on the sheet: R1
Changed lines of the file:
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@@
     (stroke (width 0) (type default))
   )
-  (wire (pts (xy 200.66 73.66) (xy 203.2 73.66))
-    (stroke (width 0) (type default))
-  )
   (wire (pts (xy 57.15 171.45) (xy 67.31 171.45))
     (stroke (width 0) (type default))
@@
     (stroke (width 0) (type default))
   )
-  (wire (pts (xy 200.66 76.2) (xy 200.66 73.66))
-    (stroke (width 0) (type default))
-  )
   (wire (pts (xy 16.51 156.21) (xy 26.67 156.21))
     (stroke (width 0) (type default))
@@
     (stroke (width 0) (type default))
   )
-  (wire (pts (xy 194.31 76.2) (xy 200.66 76.2))
-    (stroke (width 0) (type default))
-  )
   (wire (pts (xy 152.4 22.86) (xy 154.94 22.86))
     (stroke (width 0) (type default))
@@
     (stroke (width 0) (type default))
   )
-  (wire (pts (xy 184.15 81.28) (xy 191.77 81.28))
+  (wire (pts (xy 184.15 81.28) (xy 196.85 81.28))
     (stroke (width 0) (type default))
   )
@@
     (effects (font (size 1.27 1.27)) (justify left bottom))
   )
-  (label "DONE" (at 191.77 81.28 0) (fields_autoplaced)
-    (effects (font (size 1.27 1.27)) (justify left bottom))
+  (label "DONE" (at 196.85 81.28 180) (fields_autoplaced)
+    (effects (font (size 1.27 1.27)) (justify right bottom))
   )
   (label "~{C60M}" (at 210.82 130.81 180) (fields_autoplaced)
@@
       (effects (font (size 1.27 1.27)))
     )
-    (property "Value" "LCMXO2-640HC-TG100C" (at 160.02 83.82 0)
+    (property "Value" "LCMXO2-640HC-4TG100C" (at 160.02 83.82 0)
       (effects (font (size 1.016 1.016)))
     )
@@
     )
   )
-  (symbol (lib_id "Device:R_Small") (at 194.31 73.66 0) (mirror y) (unit 1)
+  (symbol (lib_id "Device:R_Small") (at 194.31 68.58 180) (unit 1)
     (in_bom yes) (on_board yes) (dnp no)
-    (property "Reference" "R1" (at 195.8086 72.4916 0)
+    (property "Reference" "R1" (at 195.58 67.31 0)
       (effects (font (size 1.27 1.27)) (justify right))
     )
-    (property "Value" "10k" (at 195.8086 74.803 0)
+    (property "Value" "10k" (at 195.58 69.85 0)
       (effects (font (size 1.27 1.27)) (justify right))
     )
-    (property "Footprint" "stdpads:R_0603" (at 194.31 73.66 0)
+    (property "Footprint" "stdpads:R_0603" (at 194.31 68.58 0)
       (effects (font (size 1.27 1.27)) hide)
     )
-    (property "Datasheet" "" (at 194.31 73.66 0)
+    (property "Datasheet" "" (at 194.31 68.58 0)
       (effects (font (size 1.27 1.27)) hide)
     )
-    (property "LCSC Part" "C25804" (at 194.31 73.66 0)
+    (property "LCSC Part" "C25804" (at 194.31 68.58 0)
       (effects (font (size 1.27 1.27)) hide)
     )
@@
     )
   )
-  (symbol (lib_id "power:GND") (at 203.2 73.66 0) (mirror y) (unit 1)
-    (in_bom yes) (on_board yes) (dnp no)
-    (property "Reference" "#PWR0159" (at 203.2 80.01 0)
-      (effects (font (size 1.27 1.27)) hide)
-    )
-    (property "Value" "GND" (at 203.2 77.47 0)
-      (effects (font (size 1.27 1.27)))
-    )
-    (property "Footprint" "" (at 203.2 73.66 0)
-      (effects (font (size 1.27 1.27)) hide)
-    )
-    (property "Datasheet" "" (at 203.2 73.66 0)
-      (effects (font (size 1.27 1.27)) hide)
-    )
-    (pin "1")
-    (instances
-      (project "RAM2GS"
-        (path "/0fd24f5c-4245-40b1-8698-6faceb999cd9"
-          (reference "#PWR0159") (unit 1)
-        )
-      )
-    )
-  )
   (symbol (lib_id "Device:R_Small") (at 127 173.99 270) (unit 1)
     (in_bom yes) (on_board yes) (dnp no)
@@
       (effects (font (size 1.27 1.27)) (justify left))
     )
-    (property "Value" "15p" (at 131.8768 178.943 0)
+    (property "Value" "22p" (at 131.8768 178.943 0)
       (effects (font (size 1.27 1.27)) (justify left))
     )
@@
         )
       )
+    )
+  )
+  (symbol (lib_id "power:+3V3") (at 194.31 66.04 0) (unit 1)
+    (in_bom yes) (on_board yes) (dnp no)
+    (property "Reference" "#PWR02" (at 194.31 69.85 0)
+      (effects (font (size 1.27 1.27)) hide)
+    )
+    (property "Value" "+3V3" (at 194.31 62.23 0)
+      (effects (font (size 1.27 1.27)))
+    )
+    (property "Footprint" "" (at 194.31 66.04 0)
+      (effects (font (size 1.27 1.27)) hide)
+    )
+    (property "Datasheet" "" (at 194.31 66.04 0)
+      (effects (font (size 1.27 1.27)) hide)
+    )
+    (pin "1")
+    (instances
+      (project "RAM2GS"
+        (path "/0fd24f5c-4245-40b1-8698-6faceb999cd9"
+          (reference "#PWR02") (unit 1)
+        )
+      )

Commit message: 2.2
Parts:
- H1, H2, H3, H4, H5: value (none) -> ~
- R2, R3: value 47 -> DNP; LCSC Part C23182 -> (none)
- U10: value 74LVC1G04GW -> DNP; LCSC Part C10237 -> (none)

Commit message: RC D.2.3
Connections:
- net +3V3: now also U1.11 ((VccIO3))
- no-connect marks 16 -> 18
Changed lines of the file:
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@@
 	(title_block
 		(title "GW4201D (RAM2GS II) - LCMXO2-640 / LCMXO2-1200")
-		(date "2024-04-24")
-		(rev "2.2")
+		(date "2025-02-14")
+		(rev "2.3")
 		(company "Garrett's Workshop")
 	)
@@
 	)
 	(junction
-		(at 170.18 22.86)
+		(at 172.72 22.86)
 		(diameter 0)
 		(color 0 0 0 0)
@@
 	)
 	(junction
-		(at 162.56 22.86)
+		(at 165.1 22.86)
 		(diameter 0)
 		(color 0 0 0 0)
@@
 	)
 	(junction
+		(at 152.4 22.86)
+		(diameter 0)
+		(color 0 0 0 0)
+	)
+	(junction
 		(at 226.06 48.26)
 		(diameter 0)
@@
 	)
 	(junction
-		(at 157.48 22.86)
+		(at 160.02 22.86)
 		(diameter 0)
 		(color 0 0 0 0)
@@
 	)
 	(junction
-		(at 154.94 22.86)
+		(at 157.48 22.86)
 		(diameter 0)
 		(color 0 0 0 0)
@@
 	)
 	(junction
-		(at 160.02 22.86)
+		(at 162.56 22.86)
 		(diameter 0)
 		(color 0 0 0 0)
@@
 	)
 	(junction
-		(at 152.4 22.86)
+		(at 154.94 22.86)
 		(diameter 0)
 		(color 0 0 0 0)
@@
 	)
 	(junction
-		(at 165.1 22.86)
+		(at 167.64 22.86)
 		(diameter 0)
 		(color 0 0 0 0)
@@
 	)
 	(no_connect
+		(at 250.19 93.98)
+	)
+	(no_connect
 		(at 101.6 184.15)
 	)
@@
 	)
 	(no_connect
+		(at 184.15 137.16)
+	)
+	(no_connect
 		(at 135.89 91.44)
 	)
@@
 	(wire
 		(pts
-			(xy 162.56 22.86) (xy 165.1 22.86)
+			(xy 165.1 22.86) (xy 167.64 22.86)
 		)
 		(stroke
@@
 	(wire
 		(pts
-			(xy 154.94 22.86) (xy 157.48 22.86)
+			(xy 157.48 22.86) (xy 160.02 22.86)
 		)
 		(stroke
@@
 	(wire
 		(pts
-			(xy 152.4 22.86) (xy 154.94 22.86)
+			(xy 154.94 22.86) (xy 157.48 22.86)
 		)
 		(stroke
@@
 	(wire
 		(pts
+			(xy 152.4 22.86) (xy 154.94 22.86)
+		)
+		(stroke
+			(width 0)
+			(type default)
+		)
+	)
+	(wire
+		(pts
 			(xy 105.41 181.61) (xy 101.6 181.61)
 		)
@@
 	(wire
 		(pts
-			(xy 172.72 22.86) (xy 170.18 22.86)
+			(xy 175.26 22.86) (xy 172.72 22.86)
 		)
 		(stroke
@@
 	(wire
 		(pts
-			(xy 165.1 22.86) (xy 167.64 22.86)
+			(xy 167.64 22.86) (xy 170.18 22.86)
 		)
 		(stroke
@@
 	(wire
 		(pts
-			(xy 157.48 22.86) (xy 160.02 22.86)
+			(xy 160.02 22.86) (xy 162.56 22.86)
 		)
 		(stroke
@@
 	(wire
 		(pts
-			(xy 160.02 22.86) (xy 162.56 22.86)
+			(xy 162.56 22.86) (xy 165.1 22.86)
 		)
 		(stroke
@@
 		(pin "9"
 		)
+		(pin "40"
+		)
 		(instances
 			(project "RAM2GS"
@@
 		(pin "99"
 		)
+		(pin "11"
+		)
+		(pin "61"
+		)
+		(pin "89"
+		)
 		(instances
 			(project "RAM2GS"
@@
 	(symbol
 		(lib_id "power:+1V2")
-		(at 170.18 22.86 0)
+		(at 172.72 22.86 0)
 		(unit 1)
 		(exclude_from_sim no)
@@
 		(dnp no)
 		(property "Reference" "#PWR0135"
-			(at 170.18 26.67 0)
+			(at 172.72 26.67 0)
 			(effects
 				(font
@@
 		)
 		(property "Value" "+1V2"
-			(at 170.18 19.05 0)
+			(at 172.72 19.05 0)
 			(effects
 				(font
@@
 		)
 		(property "Footprint" ""
-			(at 170.18 22.86 0)
+			(at 172.72 22.86 0)
 			(effects
 				(font
@@
 		)
 		(property "Datasheet" ""
-			(at 170.18 22.86 0)
+			(at 172.72 22.86 0)
 			(effects
 				(font
@@
 		)
 		(property "Description" ""
-			(at 170.18 22.86 0)
+			(at 172.72 22.86 0)
 			(effects
 				(font
