File: Hardware/MAX/RAM2GS.kicad_pcb (KiCad board)
At the start: 4 copper layers, 67.3 x 48.5 mm, 59 parts, among them J1 Memory Expansion, J2 JTAG, U1 EPM240T100C5N, U10 74LVC1G04GW, U11 AP2127K-1.8TRG1, U2 W9812G6KH-6, U3 60M, U4 74AHCT245PW, U5 74LVC245APW, U6 74LVC245APW, U7 74LVC245APW, U8 AZ1117CH-3.3TRG1, U9 74LVC1G04GW

Commit message: idk
Parts:
- removed RN1, RN2, RN3: 4x33, stdpads:R4_0402
- added R5: 47, stdpads:R_0603, F.Cu at (73.2, 108.0)
- R3: value 100 -> 47; footprint stdpads:R_0805 -> stdpads:R_0603
- moved R3 17.6 mm to (70.5, 108.0), turned to 180 degrees
Connections:
- R3 pad 2: Net-(R3-Pad2) -> /RClk
- U1 pad 89: /RD2r -> /RD2
- U1 pad 90: /RD1r -> /RD1
- U1 pad 91: /RD5r -> /RD5
- U1 pad 92: /RD4r -> /RD4
- U1 pad 95: /RD6r -> /RD6
- U1 pad 96: /RD0r -> /RD0
- U1 pad 97: /RD7r -> /RD7
- U1 pad 99: /RD3r -> /RD3
- U10 pad 4: Net-(RN1-Pad1) -> Net-(R3-Pad1)
- U4 pad 19: Net-(R3-Pad2) -> Net-(U4-Pad19)
- U9 pad 4: Net-(R3-Pad1) -> Net-(U4-Pad19)
Routing:
- net /RD4r: track 21.4 -> 0.00 mm, vias 2 -> 0
- net /RD5r: track 20.3 -> 0.00 mm, vias 2 -> 0
- net /RD7r: track 18.5 -> 0.00 mm, vias 2 -> 0
- net /RD6r: track 18.1 -> 0.00 mm, vias 2 -> 0
- net /RD2r: track 17.6 -> 0.00 mm, vias 2 -> 0
- net /RD1r: track 17.0 -> 0.00 mm, vias 2 -> 0
- net /RD4: track 20.0 -> 36.2 mm
- net /RD5: track 20.3 -> 36.3 mm
- net /RD7: track 20.8 -> 35.2 mm
- net /RD6: track 20.2 -> 33.9 mm
- net /RD2: track 19.4 -> 32.8 mm
- net /RD0r: track 13.2 -> 0.00 mm, vias 2 -> 0
- net /RD1: track 19.3 -> 31.9 mm
- net /RD3r: track 11.9 -> 0.00 mm, vias 2 -> 0
- net /RD0: track 18.6 -> 27.7 mm
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
Commit message: Generated gerbers and documenation PDFs
Parts:
- removed RN4, RN5: 4x33, stdpads:R4_0402
- added D1: White, stdpads:LED_0805, F.Cu at (71.3, 102.7)
- added R3: 47, stdpads:R_0603, F.Cu at (96.8, 115.8)
- added R7: 180, stdpads:R_0805, F.Cu at (71.3, 104.6)
- J1: value Memory Expansion -> IIgs RAM Exp.
- U1: value EPM240T100C5N -> EPM240T100
- moved R5 0.10 mm to (70.5, 108.0)
- moved R6 0.10 mm to (73.2, 108.0)
- renumbered R3 to R5, R5 to R6
Connections:
- U1 pad 88: Net-(U1-Pad88) -> /LED
- U1 pad 89: /RD2 -> /RD3
- U1 pad 91: /RD5 -> /RD4
- U1 pad 92: /RD4 -> /RD5
- U1 pad 99: /RD3 -> /RD2
- U7 pad 11: Net-(RN5-Pad4) -> /Ain9
- U7 pad 12: Net-(RN5-Pad3) -> /Ain8
- U7 pad 13: Net-(RN5-Pad2) -> /Ain6
- U7 pad 14: Net-(RN5-Pad1) -> /Ain3
- U7 pad 15: Net-(RN4-Pad4) -> /Ain4
- U7 pad 16: Net-(RN4-Pad3) -> /Ain5
- U7 pad 17: Net-(RN4-Pad2) -> /Ain7
Routing:
- net /LED: track 0.00 -> 18.0 mm
- net /RD3: track 28.1 -> 38.1 mm
- net /~CRAS~in: track 22.1 -> 13.0 mm
- net Net-(R3-Pad2): track 1.91 -> 10.4 mm
- net +1V8: track 143.8 -> 138.3 mm
- net /RD1: track 31.9 -> 36.9 mm
- net /RD0: track 27.7 -> 32.6 mm
- net /RD5: track 36.3 -> 41.0 mm
- net GND: track 182.1 -> 177.9 mm, vias 237 -> 226
- net /RD7: track 35.2 -> 39.4 mm
- net /RD6: track 33.9 -> 38.1 mm
- net /RD4: track 36.2 -> 39.8 mm
- net /Ain5: track 23.6 -> 25.8 mm
- net /Ain4: track 24.3 -> 26.4 mm
- net /Ain7: track 23.1 -> 25.2 mm
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- added copper zone on F.Cu, net +3V3
Other:
- board text added: "D20A"
