File: Hardware/MAX/RAM2GS.kicad_pcb (KiCad board)
At the start: 4 copper layers, 67.3 x 48.5 mm, 58 parts, among them J1 IIgs RAM Exp., J2 JTAG, U1 EPM240T100, U10 74LVC1G04GW, U11 AP2127K-1.8TRG1, U2 W9812G6KH-6, U3 60M, U4 74AHCT245PW, U5 74LVC245APW, U6 74LVC245APW, U7 74LVC245APW, U8 AZ1117CH-3.3TRG1, U9 74LVC1G04GW

Commit message: 2.1?
Parts:
- added G***: LOGO, LOGO, F.Cu at (67.2, 95.2)
- added G***: LOGO, LOGO, F.Cu at (87.5, 95.0)
- D1: value White -> Amber
- R7: value 180 -> 220
- turned U10 to 90 degrees
- turned U11 to 0 degrees
- turned U2 to -90 degrees
- turned U9 to -90 degrees
- renumbered H5 to H3, H3 to H5
Connections:
- net /R~CAS~ renamed /R~{CAS}
- net /R~CS~ renamed /R~{CS}
- net /R~RAS~ renamed /R~{RAS}
- net /R~WE~ renamed /R~{WE}
- net /S~CS~ renamed /S~{CS}
- net /~CCAS~ renamed /~{CCAS}
- net /~CCAS~in renamed /~{CCAS}in
- net /~CRAS~ renamed /~{CRAS}
- net /~CRAS~in renamed /~{CRAS}in
- net /~CROMSEL~ renamed /~{CROMSEL}
- net /~CSEL~ renamed /~{CSEL}
- net /~FWE~ renamed /~{FWE}
- net /~WE~in renamed /~{WE}in
- J2 pad 6: Net-(J2-Pad6) -> unconnected-(J2-Pin_6-Pad6)
- J2 pad 7: Net-(J2-Pad7) -> unconnected-(J2-Pin_7-Pad7)
- J2 pad 8: Net-(J2-Pad8) -> unconnected-(J2-Pin_8-Pad8)
- U1 pad 58: Net-(U1-Pad58) -> unconnected-(U1-IO2_58-Pad58)
- U1 pad 61: Net-(U1-Pad61) -> unconnected-(U1-IO2_61-Pad61)
- U1 pad 62: Net-(U1-Pad62) -> unconnected-(U1-IO2_62/GCLK2-Pad62)
- U1 pad 64: Net-(U1-Pad64) -> unconnected-(U1-IO2_64/GCLK3-Pad64)
- U1 pad 66: Net-(U1-Pad66) -> unconnected-(U1-IO2_66-Pad66)
- U1 pad 75: Net-(U1-Pad75) -> unconnected-(U1-IO2_75-Pad75)
- U1 pad 76: Net-(U1-Pad76) -> unconnected-(U1-IO2_76-Pad76)
- U1 pad 78: Net-(U1-Pad78) -> unconnected-(U1-IO2_78-Pad78)
- U1 pad 81: Net-(U1-Pad81) -> unconnected-(U1-IO2_81-Pad81)
- U1 pad 82: Net-(U1-Pad82) -> unconnected-(U1-IO2_82-Pad82)
- U1 pad 84: Net-(U1-Pad84) -> unconnected-(U1-IO2_84-Pad84)
- U1 pad 86: Net-(U1-Pad86) -> unconnected-(U1-IO2_86-Pad86)
- U10 pad 1: Net-(U10-Pad1) -> unconnected-(U10-NC-Pad1)
- U11 pad 4: Net-(U11-Pad4) -> unconnected-(U11-NC-Pad4)
- U9 pad 1: Net-(U9-Pad1) -> unconnected-(U9-NC-Pad1)
Routing:
- net /LED: track 18.0 -> 19.6 mm, vias 0 -> 2
- net +3V3: vias 99 -> 98
- net /FD2: vias 4 -> 3
- net GND: vias 226 -> 222
Other:
- net class Default removed
- rule pad_to_mask_clearance: 0.075 -> 0.0762
- rule solder_mask_min_width: 0.1 -> 0.127
- board text added: "D21A"
- board text added: "JLCJLCJLCJLC"
- board text removed: "4201D"
- board text removed: "8 MB RAM"
- board text removed: "D20A"
- board text removed: "GW"
- board text removed: "Garrett’s Workshop"
- board text removed: "for Apple IIgs"

Commit message: RC 2.2
Parts:
- J2: footprint Connector:Tag-Connect_TC2050-IDC-FP_2x05_P1.27mm_Vertical -> stdpads:Tag-Connect_TC2050-IDC-FP_2x05_P1.27mm_Vertical
Connections:
- J1 pad 11: +5V -> 5VC
Routing:
- net GND: track 177.9 -> 175.6 mm, vias 222 -> 221
- net +3V3: track 264.3 -> 262.8 mm
- net /RA11: track 21.0 -> 21.8 mm
Other:
- board text added: "D22A"
- board text removed: "D21A"

Commit message: RC
Parts:
- U1: value EPM240T100 -> EPM240T100C5N
Changed lines of the file:
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@@
       (polygon
         (pts
-          (xy 101.228936 100.067962)
-          (xy 104.821038 103.660064)
-          (xy 105.719064 102.762038)
-          (xy 102.126962 99.169936)
+          (xy 101.049331 100.067962)
+          (xy 104.821038 103.839669)
+          (xy 105.898669 102.762038)
+          (xy 102.126962 98.990331)
         )
       )
@@
         (effects (font (size 0.8128 0.8128) (thickness 0.2032)))
     )
-    (fp_text value "EPM240T100" (at 1.05 0) (layer "F.Fab")
+    (fp_text value "EPM240T100C5N" (at 1.05 0) (layer "F.Fab")
         (effects (font (size 0.508 0.508) (thickness 0.127)))
     )
@@
   (segment (start 82.45 112.2) (end 98.1 96.55) (width 0.15) (layer "B.Cu") (net 112))
   (segment (start 82.35 112.2) (end 82.45 112.2) (width 0.15) (layer "B.Cu") (net 112))
+  (segment (start 104.821038 103.660064) (end 105.710064 103.660064) (width 0.15) (layer "F.Cu") (net 116))
   (segment (start 98.856498 102.7) (end 98.078249 103.478249) (width 0.15) (layer "F.Cu") (net 116))
   (segment (start 81.05 111.7) (end 79.5 113.25) (width 0.15) (layer "F.Cu") (net 116))
-  (segment (start 104.821038 103.660064) (end 105.710064 103.660064) (width 0.15) (layer "F.Cu") (net 116))
   (segment (start 79.5 113.25) (end 78.9 113.25) (width 0.15) (layer "F.Cu") (net 116))
+  (segment (start 105.710064 103.660064) (end 106.4 104.35) (width 0.15) (layer "F.Cu") (net 116))
   (segment (start 78.7 113.05) (end 77.7375 113.05) (width 0.15) (layer "F.Cu") (net 116))
   (segment (start 99.6 102.9) (end 99.4 102.7) (width 0.15) (layer "F.Cu") (net 116))
   (segment (start 99.4 102.7) (end 98.856498 102.7) (width 0.15) (layer "F.Cu") (net 116))
   (segment (start 78.9 113.25) (end 78.7 113.05) (width 0.15) (layer "F.Cu") (net 116))
-  (segment (start 106.5 105.3) (end 105.7 106.1) (width 0.15) (layer "F.Cu") (net 116))
-  (segment (start 105.710064 103.660064) (end 106.5 104.45) (width 0.15) (layer "F.Cu") (net 116))
+  (segment (start 106.4 104.35) (end 106.4 105.4) (width 0.15) (layer "F.Cu") (net 116))
   (segment (start 81.4 111.7) (end 81.05 111.7) (width 0.15) (layer "F.Cu") (net 116))
-  (segment (start 106.5 104.45) (end 106.5 105.3) (width 0.15) (layer "F.Cu") (net 116))
+  (segment (start 106.4 105.4) (end 105.7 106.1) (width 0.15) (layer "F.Cu") (net 116))
   (via (at 105.7 106.1) (size 0.5) (drill 0.3) (layers "F.Cu" "B.Cu") (net 116))
   (via (at 81.4 111.7) (size 0.5) (drill 0.3) (layers "F.Cu" "B.Cu") (net 116))
@@
       )
     )
-  )
-  (zone (net 0) (net_name "") (layer "F.Cu") (hatch edge 0.508)
-    (connect_pads (clearance 0))
-    (min_thickness 0.254) (filled_areas_thickness no)
-    (keepout (tracks allowed) (vias allowed) (pads allowed) (copperpour not_allowed) (footprints allowed))
-    (fill (thermal_gap 0.508) (thermal_bridge_width 0.508))
-    (polygon
-      (pts
-        (xy 105.7219 102.76374)
-        (xy 104.82274 103.6629)
-        (xy 101.22864 100.0688)
-        (xy 102.1278 99.16964)
-      )
-    )

Commit message: 2.2
Parts:
- H1, H2, H3, H4, H5: value (none) -> ~

Commit message: RC D.2.3
Connections:
- U2 pad 40: (no net) -> unconnected-(U2-NC-Pad40)
Other:
- board text added: "D23A"
- board text removed: "D22A"
