File: Hardware/MAX/RAM2GS.sch (KiCad schematic (older format))
At the start: 59 parts, among them J1 Memory Expansion, J2 JTAG, U1 EPM240T100C5N, U10 74LVC1G04GW, U11 AP2127K-1.8TRG1, U2 W9812G6KH-6, U3 60M, U4 74AHCT245PW, U5 74LVC245APW, U6 74LVC245APW, U7 74LVC245APW, U8 AZ1117CH-3.3TRG1, U9 74LVC1G04GW

Commit message: almost done
Parts:
- U2: Mfg. Part Numbers Winbond W9812G6KH-6 Winbond W9812G6KH-6I, Winbond W9825G6KH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 -> Winbond W9812G6KH-6, Winbond W9812G6KH-6I, Winbond W9825G6K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
- U3: Notes Most 60-62.5 MHz crystal oscillator or silicon oscillator i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 -> Most 60-62.5 MHz 3.3V crystal oscillator or silicon oscilla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
Other:
- moved on the sheet: C28, R4
Changed lines of the file:
@@
 L power:+3V3 #PWR0133
 U 1 1 5E9850F8
-P 2050 3850
-F 0 "#PWR0133" H 2050 3700 50  0001 C CNN
-F 1 "+3V3" H 2050 4000 50  0000 C CNN
-F 2 "" H 2050 3850 50  0001 C CNN
-F 3 "" H 2050 3850 50  0001 C CNN
-	1    2050 3850
-	1    0    0    -1
-$EndComp
-$Comp
-L power:+5V #PWR0134
-U 1 1 5E9856CC
-P 1150 3850
-F 0 "#PWR0134" H 1150 3700 50  0001 C CNN
-F 1 "+5V" H 1150 4000 50  0000 C CNN
-F 2 "" H 1150 3850 50  0001 C CNN
-F 3 "" H 1150 3850 50  0001 C CNN
-	1    1150 3850
-	-1   0    0    -1
+P 2150 3850
+F 0 "#PWR0133" H 2150 3700 50  0001 C CNN
+F 1 "+3V3" H 2150 4000 50  0000 C CNN
+F 2 "" H 2150 3850 50  0001 C CNN
+F 3 "" H 2150 3850 50  0001 C CNN
+	1    2150 3850
+	1    0    0    -1
 $EndComp
 $Sheet
@@
 F 3 "" H 9400 2650 50  0001 C CNN
 F 4 "C62379" H 9400 2900 50  0001 C CNN "LCSC Part"
-F 5 "Winbond W9812G6KH-6 Winbond W9812G6KH-6I, Winbond W9825G6KH-6, Winbond W9825G6KH-6I, ISSI IS42S16160J-6TL, ISSI IS42S16160J-6TLI, Micron MT48LC16M16A2P-6A :G, Micron MT48LC16M16A2P-6A IT:G" H 9400 2900 50  0001 C CNN "Mfg. Part Numbers"
+F 5 "Winbond W9812G6KH-6, Winbond W9812G6KH-6I, Winbond W9825G6KH-6, Winbond W9825G6KH-6I, ISSI IS42S16160J-6TL, ISSI IS42S16160J-6TLI, Micron MT48LC16M16A2P-6A :G, Micron MT48LC16M16A2P-6A IT:G" H 9400 2900 50  0001 C CNN "Mfg. Part Numbers"
 F 6 "Most 166 MHz 128/256 Mbit SDRAM is acceptable." H 9400 2900 50  0001 C CNN "Notes"
 	1    9400 2900
@@
 U 1 1 5E9D5897
 P 6250 3300
-F 0 "U1" H 6200 5850 50  0000 C CNN
-F 1 "EPM240T100C5N" H 6200 5750 50  0000 C CNN
+F 0 "U1" H 6250 3350 50  0000 C CNN
+F 1 "EPM240T100C5N" H 6250 3250 50  0000 C CNN
 F 2 "stdpads:TQFP-100_14x14mm_P0.5mm" H 6250 3200 20  0001 C CNN
 F 3 "" H 6250 3300 50  0001 C CNN
@@
 F 4 "C26255" H 9950 5050 50  0001 C CNN "LCSC Part"
 F 5 "SiTime SIT1602AI-82-33E-60.000000Y, Shenzhen SCTF S7D60.000000B20F30T, Taiten OCETGLJTNF-60MHZ" H 9950 5050 50  0001 C CNN "Mfg. Part Numbers"
-F 6 "Most 60-62.5 MHz crystal oscillator or silicon oscillator is acceptable. Do not use crystal resonator or ceramic resonator." H 9950 5050 50  0001 C CNN "Notes"
+F 6 "Most 60-62.5 MHz 3.3V crystal oscillator or silicon oscillator is acceptable. Do not use crystal resonator or ceramic resonator." H 9950 5050 50  0001 C CNN "Notes"
 	1    9950 5050
 	-1   0    0    -1
@@
 	0    1    1    0
 $EndComp
-Wire Wire Line
-	2050 3850 1850 3850
-Wire Wire Line
-	1150 3850 1250 3850
 Connection ~ 2250 6950
 Connection ~ 2250 7350
@@
 	-1   0    0    -1
 $EndComp
-Wire Wire Line
-	1250 4650 1150 4650
-Wire Wire Line
-	1150 4650 1150 4550
-Connection ~ 1150 3850
-Wire Wire Line
-	1250 4550 1150 4550
-Connection ~ 1150 4550
-Wire Wire Line
-	1150 4550 1150 3850
 $Comp
 L Regulator_Linear:AP2127K-1.8 U11
@@
 $EndComp
 Wire Wire Line
-	1850 4550 2050 4550
+	1850 4550 1950 4550
 $Comp
 L Device:C_Small C28
 U 1 1 871B6E7B
-P 2050 4650
-F 0 "C28" H 2142 4696 50  0000 L CNN
-F 1 "2u2" H 2142 4605 50  0000 L CNN
-F 2 "stdpads:C_0603" H 2050 4650 50  0001 C CNN
-F 3 "" H 2050 4650 50  0001 C CNN
-F 4 "C23630" H 2050 4650 50  0001 C CNN "LCSC Part"
-F 5 "Samsung CL10A225KO8NNNC" H 2050 4650 50  0001 C CNN "Mfg. Part Numbers"
-F 6 "10V or higher. Any manufacturer's part is acceptable but Samsung, Murata, Yageo preferred." H 2050 4650 50  0001 C CNN "Notes"
-	1    2050 4650
-	1    0    0    -1
-$EndComp
-Wire Wire Line
-	2050 4750 2050 4950
-Wire Wire Line
-	2050 4950 1550 4950
+P 2150 4650
+F 0 "C28" H 2242 4696 50  0000 L CNN
+F 1 "2u2" H 2242 4605 50  0000 L CNN
+F 2 "stdpads:C_0603" H 2150 4650 50  0001 C CNN
+F 3 "" H 2150 4650 50  0001 C CNN
+F 4 "C23630" H 2150 4650 50  0001 C CNN "LCSC Part"
+F 5 "Samsung CL10A225KO8NNNC" H 2150 4650 50  0001 C CNN "Mfg. Part Numbers"
+F 6 "10V or higher. Any manufacturer's part is acceptable but Samsung, Murata, Yageo preferred." H 2150 4650 50  0001 C CNN "Notes"
+	1    2150 4650
+	1    0    0    -1
+$EndComp
+Wire Wire Line
+	2150 4750 2150 4950
+Wire Wire Line
+	2150 4950 1550 4950
 Connection ~ 1550 4950
 $Comp
 L power:+1V8 #PWR0160
 U 1 1 871BC45D
-P 2050 4550
-F 0 "#PWR0160" H 2050 4400 50  0001 C CNN
-F 1 "+1V8" H 2050 4700 50  0000 C CNN
-F 2 "" H 2050 4550 50  0001 C CNN
-F 3 "" H 2050 4550 50  0001 C CNN
-	1    2050 4550
-	1    0    0    -1
-$EndComp
-Connection ~ 2050 4550
+P 2150 4550
+F 0 "#PWR0160" H 2150 4400 50  0001 C CNN
+F 1 "+1V8" H 2150 4700 50  0000 C CNN
+F 2 "" H 2150 4550 50  0001 C CNN
+F 3 "" H 2150 4550 50  0001 C CNN
+	1    2150 4550
+	1    0    0    -1
+$EndComp
+Connection ~ 2150 4550
 $Comp
 L Device:R_Small R4
 U 1 1 871C5B73
-P 1850 4200
-F 0 "R4" H 1791 4246 50  0000 R CNN
-F 1 "0" H 1791 4155 50  0000 R CNN
-F 2 "stdpads:R_0805" H 1850 4200 50  0001 C CNN
-F 3 "" H 1850 4200 50  0001 C CNN
-F 4 "C17477" H 1850 4200 50  0001 C CNN "LCSC Part"
-F 5 "Uniroyal 0805W8F0000T5E" H 1850 4200 50  0001 C CNN "Mfg. Part Numbers"
-F 6 "Any manufacturer's part is acceptable." H 1850 4200 50  0001 C CNN "Notes"
-	1    1850 4200
-	-1   0    0    -1
-$EndComp
-Wire Wire Line
-	1850 4100 1850 3850
-Connection ~ 1850 3850
-Connection ~ 1850 4550
-Wire Wire Line
-	1850 4300 1850 4550
+P 1950 4200
+F 0 "R4" H 1891 4246 50  0000 R CNN
+F 1 "0" H 1891 4155 50  0000 R CNN
+F 2 "stdpads:R_0805" H 1950 4200 50  0001 C CNN
+F 3 "" H 1950 4200 50  0001 C CNN
+F 4 "C17477" H 1950 4200 50  0001 C CNN "LCSC Part"
+F 5 "Uniroyal 0805W8F0000T5E" H 1950 4200 50  0001 C CNN "Mfg. Part Numbers"
+F 6 "Any manufacturer's part is acceptable." H 1950 4200 50  0001 C CNN "Notes"
+	1    1950 4200
+	-1   0    0    -1
+$EndComp
 Wire Wire Line
 	6650 5700 6550 5700
@@
 Text Label 7250 4200 0    50   ~ 0
 S~CS~
+Wire Wire Line
+	1950 4300 1950 4550
+Connection ~ 1950 4550
+Wire Wire Line
+	1950 4550 2150 4550
+Wire Wire Line
+	1950 4100 1950 3850
+Wire Wire Line
+	2150 3850 1950 3850
+Wire Wire Line
+	1950 3850 1850 3850
+Connection ~ 1950 3850
+$Comp
+L power:+5V #PWR0134
+U 1 1 5E9856CC
+P 1050 3850
+F 0 "#PWR0134" H 1050 3700 50  0001 C CNN
+F 1 "+5V" H 1050 4000 50  0000 C CNN
+F 2 "" H 1050 3850 50  0001 C CNN
+F 3 "" H 1050 3850 50  0001 C CNN
+	1    1050 3850
+	-1   0    0    -1
+$EndComp
+Wire Wire Line
+	1050 3850 1250 3850
+Connection ~ 1050 3850
+Wire Wire Line
+	1050 4650 1050 4550
+Wire Wire Line
+	1250 4650 1050 4650
+Connection ~ 1050 4550
+Wire Wire Line
+	1250 4550 1050 4550
+Wire Wire Line
+	1050 4550 1050 3850
 $EndSCHEMATC

Commit message: idk
Parts:
- removed RN1, RN2, RN3: 4x33, stdpads:R4_0402, symbol Device:R_Pack04
- added R5: 47, stdpads:R_0603, symbol Device:R_Small
- R3: value 100 -> 47; footprint stdpads:R_0805 -> stdpads:R_0603; LCSC Part C17408 -> (none); Mfg. Part Numbers Uniroyal 0805W8F1000T5E -> (none); Notes Any manufacturer's part is acceptable. -> (none)
Connections:
- net RD0r is gone; now on net RD0: U1.96 (IO2_96)
- net RD1r is gone; now on net RD1: U1.90 (IO2_90)
- net RD2r is gone; now on net RD2: U1.89 (IO2_89)
- net RD3r is gone; now on net RD3: U1.99 (IO2_99)
- net RD4r is gone; now on net RD4: U1.92 (IO2_92)
- net RD5r is gone; now on net RD5: U1.91 (IO2_91)
- net RD6r is gone; now on net RD6: U1.95 (IO2_95)
- net RD7r is gone; now on net RD7: U1.97 (IO2_97)
- net AClk: now also R5.2
- net RClk: now also R3.2
- net at U4.19 (~OE~): now also U9.4 (Y); no longer R3.2
- net at U10.4 (Y): now also R3.1, R5.1
- no-connect marks 23 -> 19
Changed lines of the file:
@@
 Text Label 9900 3600 0    50   ~ 0
 DQMH
-$Comp
-L Device:R_Pack04 RN2
-U 1 1 5ECF18AE
-P 8100 3500
-F 0 "RN2" V 7800 3500 50  0000 C CNN
-F 1 "4x33" V 8300 3500 50  0000 C CNN
-F 2 "stdpads:R4_0402" V 8375 3500 50  0001 C CNN
-F 3 "" H 8100 3500 50  0001 C CNN
-F 4 "C25501" H 8100 3500 50  0001 C CNN "LCSC Part"
-F 5 "Any manufacturer's part is acceptable." H 8100 3500 50  0001 C CNN "Notes"
-F 6 "Uniroyal 4D02WGJ0330TCE" H 8100 3500 50  0001 C CNN "Mfg. Part Numbers"
-	1    8100 3500
-	0    1    1    0
-$EndComp
-$Comp
-L Device:R_Pack04 RN3
-U 1 1 5ECF28B3
-P 8100 4100
-F 0 "RN3" V 7800 4100 50  0000 C CNN
-F 1 "4x33" V 8300 4100 50  0000 C CNN
-F 2 "stdpads:R4_0402" V 8375 4100 50  0001 C CNN
-F 3 "" H 8100 4100 50  0001 C CNN
-F 4 "C25501" H 8100 4100 50  0001 C CNN "LCSC Part"
-F 5 "Any manufacturer's part is acceptable." H 8100 4100 50  0001 C CNN "Notes"
-F 6 "Uniroyal 4D02WGJ0330TCE" H 8100 4100 50  0001 C CNN "Mfg. Part Numbers"
-	1    8100 4100
-	0    1    1    0
-$EndComp
-Text Label 7900 3300 2    50   ~ 0
-RD0
-Text Label 7900 3400 2    50   ~ 0
-RD1
-Text Label 7900 3500 2    50   ~ 0
-RD2
-Text Label 7900 3600 2    50   ~ 0
-RD3
-Text Label 7900 3900 2    50   ~ 0
-RD4
-Text Label 7900 4000 2    50   ~ 0
-RD5
-Text Label 7900 4100 2    50   ~ 0
-RD6
-Text Label 7900 4200 2    50   ~ 0
-RD7
-Text Label 8300 3400 0    50   ~ 0
-RD1r
-Text Label 8300 3500 0    50   ~ 0
-RD2r
-Text Label 8300 3600 0    50   ~ 0
-RD3r
-Text Label 8300 3900 0    50   ~ 0
-RD4r
-Text Label 8300 4000 0    50   ~ 0
-RD5r
-Text Label 8300 4100 0    50   ~ 0
-RD6r
-Text Label 8300 4200 0    50   ~ 0
-RD7r
-Text Label 8300 3300 0    50   ~ 0
-RD0r
 Text Label 9900 3900 0    50   ~ 0
 R~CS~
@@
 Ain9
 Text Label 7250 4500 0    50   ~ 0
-RD1r
+RD1
 Text Label 7250 4400 0    50   ~ 0
-RD2r
+RD2
 Text Label 7250 5200 0    50   ~ 0
-RD3r
+RD3
 Text Label 7250 4700 0    50   ~ 0
-RD4r
+RD4
 Text Label 7250 4600 0    50   ~ 0
-RD5r
+RD5
 Text Label 7250 4800 0    50   ~ 0
-RD6r
+RD6
 Text Label 7250 5000 0    50   ~ 0
-RD7r
-Text Label 7250 4900 0    50   ~ 0
-RD0r
+RD7
 Text Label 7250 5100 0    50   ~ 0
 DQML
@@
 	-1   0    0    -1
 $EndComp
-Text Label 8300 5150 2    50   ~ 0
+Text Label 8500 5150 2    50   ~ 0
 AClk
-$Comp
-L Device:R_Pack04 RN1
-U 1 1 5E97937D
-P 8500 5050
-F 0 "RN1" V 8200 5050 50  0000 C CNN
-F 1 "4x33" V 8700 5050 50  0000 C CNN
-F 2 "stdpads:R4_0402" V 8775 5050 50  0001 C CNN
-F 3 "" H 8500 5050 50  0001 C CNN
-F 4 "C25501" H 8500 5050 50  0001 C CNN "LCSC Part"
-F 5 "Any manufacturer's part is acceptable." H 8500 5050 50  0001 C CNN "Notes"
-F 6 "Uniroyal 4D02WGJ0330TCE" H 8500 5050 50  0001 C CNN "Mfg. Part Numbers"
-	1    8500 5050
-	0    -1   1    0
-$EndComp
-Text Label 8300 4850 2    50   ~ 0
+Text Label 8500 4850 2    50   ~ 0
 RClk
 $Comp
@@
 Wire Wire Line
 	6450 5700 6550 5700
-NoConn ~ 8300 4950
-NoConn ~ 8300 5050
 Wire Wire Line
 	8750 5150 8750 4850
@@
 Wire Wire Line
 	8750 5150 8800 5150
-NoConn ~ 8700 4950
-NoConn ~ 8700 5050
 Text Label 4900 1050 0    50   ~ 0
 ~CSEL~
@@
 Wire Wire Line
 	2150 3550 2650 3550
-$Comp
-L Device:R_Small R3
-U 1 1 5F2CC469
-P 4000 1150
-F 0 "R3" V 3950 1150 50  0000 C BNN
-F 1 "100" V 4000 1150 40  0000 C CNN
-F 2 "stdpads:R_0805" H 4000 1150 50  0001 C CNN
-F 3 "" H 4000 1150 50  0001 C CNN
-F 4 "C17408" V 4000 1150 50  0001 C CNN "LCSC Part"
-F 5 "Uniroyal 0805W8F1000T5E" H 4000 1150 50  0001 C CNN "Mfg. Part Numbers"
-F 6 "Any manufacturer's part is acceptable." H 4000 1150 50  0001 C CNN "Notes"
-	1    4000 1150
-	0    1    1    0
-$EndComp
 Connection ~ 2250 6950
 Connection ~ 2250 7350
@@
 Wire Wire Line
 	1050 4550 1050 3850
+Wire Wire Line
+	4100 1150 3900 1150
+$Comp
+L Device:R_Small R3
+U 1 1 60F771C1
+P 8600 4850
+F 0 "R3" V 8404 4850 50  0000 C CNN
+F 1 "47" V 8495 4850 50  0000 C CNN
+F 2 "stdpads:R_0603" H 8600 4850 50  0001 C CNN
+F 3 "~" H 8600 4850 50  0001 C CNN
+	1    8600 4850
+	0    1    1    0
+$EndComp
+$Comp
+L Device:R_Small R5
+U 1 1 60F76863
+P 8600 5150
+F 0 "R5" V 8404 5150 50  0000 C CNN
+F 1 "47" V 8495 5150 50  0000 C CNN
+F 2 "stdpads:R_0603" H 8600 5150 50  0001 C CNN
+F 3 "~" H 8600 5150 50  0001 C CNN
+	1    8600 5150
+	0    1    1    0
+$EndComp
+Text Label 7250 4900 0    50   ~ 0
+RD0
 $EndSCHEMATC

Commit message: Generated gerbers and documenation PDFs
Parts:
- removed RN4, RN5: 4x33, stdpads:R4_0402, symbol Device:R_Pack04
- added D1: White, stdpads:LED_0805, symbol Device:LED_Small_ALT
- added R6: 47, stdpads:R_0603, symbol Device:R_Small
- added R7: 180, stdpads:R_0805, symbol Device:R_Small
- J1: value Memory Expansion -> IIgs RAM Exp.
- R3, R5: LCSC Part (none) -> C23182; Mfg. Part Numbers (none) -> Uniroyal 0603WAF470JT5E; Notes (none) -> Any manufacturer's part is acceptable.
- U1: value EPM240T100C5N -> EPM240T100
- U10, U9: Mfg. Part Numbers NXP 74LVC1G04GW, TI SN74LVC1G04DCK -> NXP 74LVC1G04GW, TI SN74LVC1G04DCK, NXP 74AHC1G04GW, TI SN7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; Notes (none) -> Most 74LVC1G04 or 74AHC1G04 in SOT-353 package is acceptabl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
- U11: Notes (none) -> Most 1.8V regulator in SOT-23-5 package is acceptable.
- U2: Notes Most 166 MHz 128/256 Mbit SDRAM is acceptable. -> Most 166 MHz 128/256 Mbit x16 SDRAM is acceptable.
- U4: Mfg. Part Numbers NXP 74AHCT245PW, TI SN74AHCT245PW -> NXP 74AHCT245PW, NXP 74AHCT245APW, TI SN74AHCT245PW; Notes (none) -> Most 74AHCT245 in TSSOP-20 package is acceptable.
- U5, U6, U7: Mfg. Part Numbers NXP 74LVC245APW, TI SN74LVC245APW -> NXP 74LVC245APW, TI SN74LVC245APW, NXP 74AHC245PW, NXP 74AH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; Notes (none) -> Most 74LVC245 or 74AHC245 in TSSOP-20 package is acceptable.
Connections:
- net +3V3: now also R7.2
- net AClk: now also R6.2; no longer R5.2
- net Ain3: now also U7.14 (B4)
- net Ain4: now also U7.15 (B3)
- net Ain5: now also U7.16 (B2)
- net Ain6: now also U7.13 (B5)
- net Ain7: now also U7.17 (B1)
- net Ain8: now also U7.12 (B6)
- net Ain9: now also U7.11 (B7)
- net RClk: now also R5.2; no longer R3.2
- net RD2: now also U1.99 (IO2_99); no longer U1.89 (IO2_89)
- net RD3: now also U1.89 (IO2_89); no longer U1.99 (IO2_99)
- net RD4: now also U1.91 (IO2_91); no longer U1.92 (IO2_92)
- net RD5: now also U1.92 (IO2_92); no longer U1.91 (IO2_91)
- net ~CRAS~in: now also R3.1
- net at U7.18 (B0): now also R3.2
- net LED: now reaches U1.88 (IO2_88)
- net LED: now also D1.1 (K)
- net at R5.1, U10.4 (Y): now also R6.1; no longer R3.1
- new net: D1.2 (A), R7.1
- no-connect marks 19 -> 18

Commit message: BOM fixes
Parts:
- U1: Mfg. Part Numbers Altera EPM240T100C5N, Altera EPM240T100C4N, Altera EPM240T1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 -> Altera 5M240ZT100C5N, Altera 5M240ZT100C4N, Altera 5M240ZT1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
Changed lines of the file:
@@
 F 3 "" H 6250 3300 50  0001 C CNN
 F 4 "C10041" H 6250 3300 50  0001 C CNN "LCSC Part"
-F 5 "Altera EPM240T100C5N, Altera EPM240T100C4N, Altera EPM240T100C3N, Altera EPM240T100I5N, Altera EPM240T100I4N, Altera EPM240T100A5N, Altera EPM240T100A4N, AGM/Alta-Gate AG256SL100, AGM AG256SL100C3, AGM AG256SL100C4, AGM/Alta-Gate AG272SL100, AGM AG272SL100C3, AGM AG272SL100C4, AGM/Alta-Gate AG576SL100, AGM AG576SL100C3, AGM AG576SL100C4" H 6250 3300 50  0001 C CNN "Mfg. Part Numbers"
+F 5 "Altera 5M240ZT100C5N, Altera 5M240ZT100C4N, Altera 5M240ZT100C3N, Altera 5M240ZT100I5N, Altera 5M240ZT100I4N, Altera 5M240ZT100A5N, Altera 5M240ZT100A4N, Altera EPM240T100C5N, Altera EPM240T100C4N, Altera EPM240T100C3N, Altera EPM240T100I5N, Altera EPM240T100I4N, Altera EPM240T100A5N, Altera EPM240T100A4N, AGM/Alta-Gate AG256SL100, AGM AG256SL100C3, AGM AG256SL100C4, AGM/Alta-Gate AG272SL100, AGM AG272SL100C3, AGM AG272SL100C4, AGM/Alta-Gate AG576SL100, AGM AG576SL100C3, AGM AG576SL100C4" H 6250 3300 50  0001 C CNN "Mfg. Part Numbers"
 	1    6250 3300
 	1    0    0    -1
