File: Hardware/iCE40/RAM2GS.kicad_pcb (KiCad board)
At the start: 4 copper layers, 67.3 x 48.5 mm, 65 parts, among them J1 Memory Expansion, J2 JTAG, U1 iCE40HX1K-TQFP-100, U10 74LVC1G04GW, U11 SPIFlash-SON-8-1EP, U12 AP2127K-1.2, U13 AP2127K-2.5, U2 W9812G6KH-6, U3 60M, U4 74AHCT245PW, U5 74LVC245APW, U6 74LVC245APW, U7 74LVC245APW, U8 AZ1117CH-3.3, U9 74LVC1G04GW

Commit message: finished MAX, LCMXO, iCE40?
Parts:
- removed R4: 0, stdpads:R_0805
- added C34: 2u2, stdpads:C_0603, F.Cu at (71.4, 99.3)
- added R5: DNP, stdpads:R_0805, F.Cu at (47.7, 126.0)
- added RN6: 4x10k, stdpads:R4_0402, F.Cu at (49.3, 123.0)
- U1: value iCE40HX1K-TQFP-100 -> iCE40HX1K-VQ100
- U11: renamed from U12; value AP2127K-1.2 -> AP2127K-1.2TRG1
- U12: renamed from U11; value SPIFlash-SON-8-1EP -> 25F010; footprint stdpads:SON-8-1EP_3x2mm_P0.5mm_EP0.25x1.65mm -> stdpads:SOIC-8_3.9mm
- U13: value AP2127K-2.5 -> AP2127K-2.5TRG1
- U8: value AZ1117CH-3.3 -> AZ1117CH-3.3TRG1
- moved FID4 8.58 mm to (58.8, 125.9)
- moved C33 0.84 mm to (60.6, 124.0)
- moved U12 0.73 mm to (53.1, 127.6), turned to 270 degrees
- moved C14 0.07 mm to (75.7, 106.8)
- renumbered RN6 to RN7
Connections:
- U12 pad 3: /D2 -> +3V3
- U12 pad 7: /D3 -> /~HOLD~
Routing:
- net +1V2: track 83.8 -> 57.2 mm, vias 6 -> 5
- net /~HOLD~: track 0.00 -> 10.8 mm
- net +2V5: track 103.1 -> 113.3 mm
- net +3V3: track 268.4 -> 272.7 mm, vias 108 -> 112
- net /D3: track 1.75 -> 0.00 mm, vias 1 -> 0
- net /D2: track 1.75 -> 0.00 mm, vias 1 -> 0
- net /C~CS~: track 44.9 -> 43.7 mm
- net /MISO: track 81.4 -> 82.5 mm
- net /S~CS~: track 83.1 -> 82.4 mm
- net /MOSI: track 84.7 -> 83.9 mm, vias 2 -> 3
- net /SCK: track 79.1 -> 79.7 mm, vias 2 -> 3
- net /CDO: track 31.2 -> 30.7 mm
- net GND: track 194.6 -> 194.9 mm, vias 227 -> 229

Commit message: almost done
Parts:
- removed R5: DNP, stdpads:R_0805
- RN6: value 4x10k -> 4x33
- moved RN6 0.43 mm to (49.0, 123.2)
Connections:
- RN6 pad 1: GND -> /CDIr
- RN6 pad 2: /MOSI -> /CDOr
- RN6 pad 3: /~HOLD~ -> /C~CS~r
- RN6 pad 4: /SCK -> /CCKr
- RN6 pad 5: +3V3 -> /CCK
- RN6 pad 6: +3V3 -> /C~CS~
- RN6 pad 7: +3V3 -> /CDO
- RN6 pad 8: GND -> /CDI
- RN7 pad 2: GND -> /CDONE
- RN7 pad 7: GND -> +3V3
- U1 pad 79: /S~CS~ -> Net-(U1-Pad79)
- U1 pad 80: /MISO -> Net-(U1-Pad80)
- U1 pad 81: /MOSI -> Net-(U1-Pad81)
- U1 pad 83: /SCK -> Net-(U1-Pad83)
- U12 pad 1: /S~CS~ -> /C~CS~r
- U12 pad 2: /MISO -> /CDIr
- U12 pad 5: /MOSI -> /CDOr
- U12 pad 6: /SCK -> /CCKr
- U12 pad 7: /~HOLD~ -> +3V3
- U13 pad 3: +5V -> +3V3
Routing:
- net /CDI: track 29.5 -> 132.6 mm, vias 2 -> 3
- net /CDO: track 30.7 -> 122.9 mm, vias 2 -> 3
- net /MOSI: track 83.9 -> 0.00 mm, vias 3 -> 0
- net /MISO: track 82.5 -> 0.00 mm, vias 2 -> 0
- net /S~CS~: track 82.4 -> 0.00 mm, vias 2 -> 0
- net /SCK: track 79.7 -> 0.00 mm, vias 3 -> 0
- net /C~CS~: track 43.7 -> 119.8 mm, vias 3 -> 4
- net /CCK: track 38.2 -> 108.7 mm, vias 2 -> 3
- net /CDONE: track 0.00 -> 23.0 mm, vias 0 -> 2
- net /CDOr: track 0.00 -> 11.3 mm
- net /~HOLD~: track 10.8 -> 0.00 mm
- net /CCKr: track 0.00 -> 8.50 mm
- net /CDIr: track 0.00 -> 5.08 mm
- net /C~CS~r: track 0.00 -> 3.61 mm
- net +5V: track 205.9 -> 207.1 mm
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
Commit message: more
Parts:
- removed RN6: 4x33, stdpads:R4_0402
- removed RN7: 4x10k, stdpads:R4_0402
- added R1: 33, stdpads:R_0603, F.Cu at (100.9, 120.3)
- added R2: 33, stdpads:R_0603, F.Cu at (51.3, 124.0)
- added R4: 33, stdpads:R_0603, F.Cu at (95.7, 117.2)
- added R5: 33, stdpads:R_0603, F.Cu at (48.3, 123.2)
- added R6: 33, stdpads:R_0603, F.Cu at (50.5, 121.8)
Connections:
- U12 pad 1: /C~CS~r -> /C~CS~
- U12 pad 2: /CDIr -> /CDI
- U12 pad 5: /CDOr -> /CDO
Routing:
- net /CDONE: track 23.0 -> 41.0 mm, vias 2 -> 4
- net /C~RST~: track 34.6 -> 49.6 mm, vias 3 -> 5
- net /CDO: track 122.9 -> 135.2 mm
- net /CDOr: track 11.3 -> 0.00 mm
- net +3V3: track 273.5 -> 281.1 mm
- net /CDI: track 132.6 -> 138.7 mm
- net /C~CS~: track 119.8 -> 125.1 mm
- net /CDIr: track 5.08 -> 0.00 mm
- net /C~CS~r: track 3.61 -> 0.00 mm
- net /CROWin1: track 16.1 -> 19.2 mm
- net /CCK: track 108.7 -> 111.6 mm
- net /CCKr: track 8.50 -> 6.73 mm
- net /Din7: track 13.0 -> 11.3 mm
- net /CROWin0: track 12.4 -> 13.9 mm
- net GND: vias 230 -> 225

Commit message: Generated gerbers and documenation PDFs
Parts:
- removed RN1, RN2, RN3, RN4, RN5: 4x33, stdpads:R4_0402
- added C35: 15p, stdpads:C_0603, F.Cu at (96.5, 101.9)
- added D1: White, stdpads:LED_0805, F.Cu at (71.3, 102.7)
- added R10: 47, stdpads:R_0603, F.Cu at (98.6, 104.0)
- added R7: 180, stdpads:R_0805, F.Cu at (71.3, 104.6)
- added R8: 47, stdpads:R_0603, F.Cu at (70.5, 108.0)
- added R9: 47, stdpads:R_0603, F.Cu at (73.2, 108.0)
- J1: value Memory Expansion -> IIgs RAM Exp.
- R1: renamed from R4; value 33 -> 10k
- R2: value 33 -> 47
- R3: value 100 -> 47; footprint stdpads:R_0805 -> stdpads:R_0603
- R4: renamed from R1; value 33 -> 10k
- R5, R6: value 33 -> 10k
- moved R3 26.4 mm to (96.8, 117.2), turned to 270 degrees
- moved R1 0.36 mm to (95.3, 117.2)
Connections:
- J2 pad 1: /CCK -> /CCKr2
- R1 pad 2: /CDONE -> /C~RST~
- R3 pad 1: Net-(R3-Pad1) -> /~CRAS~in
- R4 pad 2: /C~RST~ -> /CDONE
- U1 pad 100: /RD2r -> /RD3
- U1 pad 82: Net-(U1-Pad82) -> /LED
- U1 pad 85: /RD0r -> /RD0
- U1 pad 86: /RD3r -> /RD2
- U1 pad 87: /RD5r -> /RD4
- U1 pad 89: /RD4r -> /RD5
- U1 pad 90: /RD6r -> /RD6
- U1 pad 91: /RD7r -> /RD7
- U1 pad 99: /RD1r -> /RD1
- U4 pad 19: Net-(R3-Pad2) -> Net-(U4-Pad19)
- U7 pad 11: Net-(RN5-Pad4) -> /Ain9
- U7 pad 12: Net-(RN5-Pad3) -> /Ain8
- U7 pad 13: Net-(RN5-Pad2) -> /Ain6
- U7 pad 14: Net-(RN5-Pad1) -> /Ain3
- U7 pad 15: Net-(RN4-Pad4) -> /Ain4
- U7 pad 16: Net-(RN4-Pad3) -> /Ain5
- U7 pad 17: Net-(RN4-Pad2) -> /Ain7
- U7 pad 18: Net-(RN4-Pad1) -> Net-(R3-Pad2)
- U9 pad 4: Net-(R3-Pad1) -> Net-(U4-Pad19)
Routing:
- net /RD0: track 18.6 -> 42.3 mm
- net /CDONE: track 41.0 -> 17.8 mm, vias 4 -> 2
- net /RD0r: track 22.2 -> 0.00 mm, vias 2 -> 0
- net /RD5r: track 21.5 -> 0.00 mm, vias 2 -> 0
- net /LED: track 0.00 -> 21.3 mm
- net /RD4: track 20.0 -> 41.0 mm
- net /RD4r: track 20.7 -> 0.00 mm, vias 2 -> 0
- net /RD7: track 20.8 -> 41.3 mm
- net /RD2: track 19.4 -> 39.6 mm
- net /RD5: track 20.3 -> 40.3 mm
- net /RD3r: track 19.6 -> 0.00 mm, vias 2 -> 0
- net /RD7r: track 19.4 -> 0.00 mm, vias 2 -> 0
- net /RD6: track 20.2 -> 39.2 mm
- net /RD6r: track 18.2 -> 0.00 mm, vias 2 -> 0
- net /RD1: track 19.3 -> 32.6 mm
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Other:
- board text added: "D20D"
