File: Hardware/iCE40/RAM2GS.sch (KiCad schematic (older format))
At the start: 65 parts, among them J1 Memory Expansion, J2 JTAG, U1 iCE40HX1K-TQFP-100, U10 74LVC1G04GW, U11 SPIFlash-SON-8-1EP, U12 AP2127K-1.2, U13 AP2127K-2.5, U2 W9812G6KH-6, U3 60M, U4 74AHCT245PW, U5 74LVC245APW, U6 74LVC245APW, U7 74LVC245APW, U8 AZ1117CH-3.3, U9 74LVC1G04GW

Commit message: finished MAX, LCMXO, iCE40?
Parts:
- removed R4: 0, stdpads:R_0805, symbol Device:R_Small
- added C34: 2u2, stdpads:C_0603, symbol Device:C_Small
- added R5: DNP, stdpads:R_0805, symbol Device:R_Small
- added RN6: 4x10k, stdpads:R4_0402, symbol Device:R_Pack04
- C1, C2, C26, C3, C4: Mfg. Part Numbers (none) -> Samsung CL21A106KAYNNNE; Notes 10V or higher -> 10V or higher. Any manufacturer's part is acceptable but Sa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
- C10, C11, C12, C13, C14, C15, C16, C17, C18, C19, C20, C21, C22, C23, C24, C25, C27, C28, C29, C30, C31, C32, C33, C5, C6, C7, C8, C9: Mfg. Part Numbers (none) -> Samsung CL10A225KO8NNNC; Notes 10V or higher -> 10V or higher. Any manufacturer's part is acceptable but Sa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
- R3: Mfg. Part Numbers (none) -> Uniroyal 0805W8F1000T5E; Notes Any manufacturer's part is acceptable -> Any manufacturer's part is acceptable.
- RN1, RN2, RN3, RN4, RN5: Mfg. Part Numbers (none) -> Uniroyal 4D02WGJ0330TCE; Notes Any manufacturer's part is acceptable -> Any manufacturer's part is acceptable.
- RN7: renamed from RN6; Mfg. Part Numbers (none) -> Uniroyal 4D02WGJ0103TCE; Notes Any manufacturer's part is acceptable -> Any manufacturer's part is acceptable.
- U1: value iCE40HX1K-TQFP-100 -> iCE40HX1K-VQ100; symbol GW_PLD:iCE40HX1K-TQFP-100 -> GW_PLD:iCE40HX1K-VQ100; LCSC Part (none) -> C1519043; Mfg. Part Numbers (none) -> Lattice iCE40HX1K-VQ100
- U10, U9: Mfg. Part Numbers NXP 74LVC1G04GW TI SN74LVC1G04DCK -> NXP 74LVC1G04GW, TI SN74LVC1G04DCK
- U11: renamed from U12; value AP2127K-1.2 -> AP2127K-1.2TRG1; LCSC Part (none) -> C151376; Mfg. Part Numbers (none) -> Diodes AP2127K-1.2TRG1, Torex XC6228D122VR
- U12: renamed from U11; value SPIFlash-SON-8-1EP -> 25F010; footprint stdpads:SON-8-1EP_3x2mm_P0.5mm_EP0.25x1.65mm -> stdpads:SOIC-8_3.9mm; symbol GW_RAM:SPIFlash-SON-8-1EP -> GW_RAM:SPIFlash-SO-8; LCSC Part (none) -> C2687406; Mfg. Part Numbers (none) -> Zetta ZD25WD20BTIGT, Adesto AT25SF081-SSHD, Winbond W25X20C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; Notes (none) -> Most SPI flash in SOIC-8 (3.9mm / 150 mil width) package is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
- U13: value AP2127K-2.5 -> AP2127K-2.5TRG1; LCSC Part (none) -> C460326; Mfg. Part Numbers (none) -> Diodes AP2127K-2.5TRG1, Torex XC6206J252MR
- U2: Notes Most 166 MHz 128/256 Mbit SDRAM will work -> Most 166 MHz 128/256 Mbit SDRAM is acceptable.
- U3: Mfg. Part Numbers SiTime SIT1602AI-82-33E-60.000000Y -> SiTime SIT1602AI-82-33E-60.000000Y, Shenzhen SCTF S7D60.000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; Notes Most 60-64 MHz crystal oscillator or silicon oscillator wil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 -> Most 60-62.5 MHz crystal oscillator or silicon oscillator i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
- U4: Mfg. Part Numbers NXP 74AHCT245PW TI SN74AHCT245PW -> NXP 74AHCT245PW, TI SN74AHCT245PW
- U5, U6, U7: Mfg. Part Numbers NXP 74LVC245APW TI SN74LVC245APW -> NXP 74LVC245APW, TI SN74LVC245APW
- U8: value AZ1117CH-3.3 -> AZ1117CH-3.3TRG1; Mfg. Part Numbers Diodes AZ1117CH-3.3TR1G Diodes AZ1117EH-3.3TR1G -> Diodes AZ1117CH-3.3TRG1, Diodes AZ1117EH-3.3TRG1; Notes (none) -> Most 1117-type 3.3V regulator in SOT-223 package is accepta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
Connections:
- net D2 is gone; now on net +3V3: U12.3 (~WP~/IO2)
- net +3V3: now also C34.1, RN6.5 (R4.2), RN6.6 (R3.2), RN6.7 (R2.2)
- net GND: now also C34.2, R5.2, RN6.1 (R1.1), RN6.8 (R1.2); no longer U12.9 (GND)
- net MOSI: now also RN6.2 (R2.1)
- net SCK: now also RN6.4 (R4.1)
- net D3 renamed ~HOLD~
- net ~HOLD~: now also R5.1, RN6.3 (R3.1)
Other:
- moved on the sheet: C28, FID1, FID2, FID3, FID4, H1, H2, H3, H4, H5, J2, RN1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

Commit message: almost done
Parts:
- removed R5: DNP, stdpads:R_0805, symbol Device:R_Small
- RN6: value 4x10k -> 4x33
- U2: Mfg. Part Numbers Winbond W9812G6KH-6 Winbond W9812G6KH-6I, Winbond W9825G6KH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 -> Winbond W9812G6KH-6, Winbond W9812G6KH-6I, Winbond W9825G6K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
- U3: Notes Most 60-62.5 MHz crystal oscillator or silicon oscillator i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 -> Most 60-62.5 MHz 3.3V crystal oscillator or silicon oscilla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
Connections:
- net +3V3: now also RN7.7 (R2.2), U12.7 (~HLD~/IO3), U13.3 (EN); no longer RN6.5 (R4.2), RN6.6 (R3.2), RN6.7 (R2.2)
- net +5V: no longer U13.3 (EN)
- net CCK: now also RN6.5 (R4.2)
- net CDI: now also RN6.8 (R1.2)
- net CDO: now also RN6.7 (R2.2)
- net CDONE: now also RN7.2 (R2.1)
- net C~CS~: now also RN6.6 (R3.2)
- net GND: no longer RN6.1 (R1.1), RN6.8 (R1.2), RN7.2 (R2.1), RN7.7 (R2.2)
- net MISO: no longer names the net of U1.80 (IOT_75)
- net MISO: no longer U12.2 (DO/IO1)
- net MOSI renamed CDOr
- net CDOr: no longer U1.81 (IOT_77)
- net SCK renamed CCKr
- net CCKr: no longer U1.83 (IOT_79)
- net S~CS~: no longer names the net of U1.79 (IOT_74)
- net S~CS~: no longer U12.1 (~CS~)
- net ~HOLD~ renamed C~CS~r
- net C~CS~r: now also U12.1 (~CS~); no longer U12.7 (~HLD~/IO3)
- new net CDIr: RN6.1 (R1.1), U12.2 (DO/IO1)
- no-connect marks 10 -> 14
Other:
- moved on the sheet: C28, RN6

Commit message: more
Parts:
- removed RN6: 4x33, stdpads:R4_0402, symbol Device:R_Pack04
- removed RN7: 4x10k, stdpads:R4_0402, symbol Device:R_Pack04
- added R1, R2, R4, R5, R6: 33, stdpads:R_0603, symbol Device:R_Small
Connections:
- net CDIr is gone; now on net CDI: U12.2 (DO/IO1)
- net CDOr is gone; now on net CDO: U12.5 (DI/IO0)
- net C~CS~r is gone; now on net C~CS~: U12.1 (~CS~)
- net +3V3: now also R1.1, R4.1, R5.1, R6.1
- net CCK: now also R2.2, R6.2
- net CCKr: now also R2.1
- net CDONE: now also R4.2
- net C~CS~: now also R5.2
- net C~RST~: now also R1.2
Changed lines of the file:
@@
 Connection ~ 3050 7750
 Connection ~ 2650 7350
-$Comp
-L Device:R_Pack04 RN7
-U 1 1 614034CA
-P 5700 6400
-F 0 "RN7" V 5400 6400 50  0000 C CNN
-F 1 "4x10k" V 5900 6400 50  0000 C CNN
-F 2 "stdpads:R4_0402" V 5975 6400 50  0001 C CNN
-F 3 "" H 5700 6400 50  0001 C CNN
-F 4 "C25725" H 5700 6400 50  0001 C CNN "LCSC Part"
-F 5 "Any manufacturer's part is acceptable." H 5700 6400 50  0001 C CNN "Notes"
-F 6 "Uniroyal 4D02WGJ0103TCE" H 5700 6400 50  0001 C CNN "Mfg. Part Numbers"
-	1    5700 6400
-	0    1    1    0
-$EndComp
-$Comp
-L power:+3V3 #PWR0169
-U 1 1 6140B7B1
-P 5400 6500
-F 0 "#PWR0169" H 5400 6350 50  0001 C CNN
-F 1 "+3V3" H 5400 6650 50  0000 C CNN
-F 2 "" H 5400 6500 50  0001 C CNN
-F 3 "" H 5400 6500 50  0001 C CNN
-	1    5400 6500
-	1    0    0    -1
-$EndComp
-Wire Wire Line
-	5500 6500 5400 6500
-Wire Wire Line
-	5500 6400 5500 6500
-Connection ~ 5500 6500
-Text Label 5900 6500 0    50   ~ 0
+Text Label 5500 6950 2    50   ~ 0
 CCK
-Text Label 5900 6400 0    50   ~ 0
+Text Label 5500 6700 2    50   ~ 0
 C~CS~
 Connection ~ 6800 5700
@@
 NoConn ~ 7450 2800
 NoConn ~ 7450 3200
-$Comp
-L power:+3V3 #PWR0153
-U 1 1 6140B25C
-P 5900 6200
-F 0 "#PWR0153" H 5900 6050 50  0001 C CNN
-F 1 "+3V3" H 5900 6350 50  0000 C CNN
-F 2 "" H 5900 6200 50  0001 C CNN
-F 3 "" H 5900 6200 50  0001 C CNN
-	1    5900 6200
-	1    0    0    -1
-$EndComp
-Text Label 5500 6200 2    50   ~ 0
-C~RST~
 $Comp
 L Regulator_Linear:LD1117S33TR_SOT223 U8
@@
 $EndComp
 Connection ~ 3050 6550
-$Comp
-L Device:R_Pack04 RN6
-U 1 1 60E88DC4
-P 9900 6300
-F 0 "RN6" V 10100 6300 50  0000 C CNN
-F 1 "4x33" V 9600 6300 50  0000 C CNN
-F 2 "stdpads:R4_0402" V 10175 6300 50  0001 C CNN
-F 3 "" H 9900 6300 50  0001 C CNN
-F 4 "C25725" H 9900 6300 50  0001 C CNN "LCSC Part"
-F 5 "Any manufacturer's part is acceptable." H 9900 6300 50  0001 C CNN "Notes"
-F 6 "Uniroyal 4D02WGJ0103TCE" H 9900 6300 50  0001 C CNN "Mfg. Part Numbers"
-	1    9900 6300
-	0    1    1    0
-$EndComp
-Text Label 5500 6300 2    50   ~ 0
+Text Label 5500 6450 2    50   ~ 0
 CDONE
 Wire Wire Line
@@
 $EndComp
 Text Label 9100 6400 0    50   ~ 0
-CDOr
+CDO
 Text Label 8000 6200 2    50   ~ 0
-CDIr
+CDI
 Text Label 9100 6300 0    50   ~ 0
 CCKr
 Text Label 8000 6100 2    50   ~ 0
-C~CS~r
+C~CS~
 Wire Wire Line
 	1050 4500 1050 5250
@@
 Wire Wire Line
 	850  4600 1250 4600
-Text Label 9700 6300 2    50   ~ 0
-C~CS~r
-Text Label 9700 6200 2    50   ~ 0
-CDOr
+Text Label 9900 6400 0    50   ~ 0
+CCKr
 Text Label 9700 6400 2    50   ~ 0
-CCKr
-Text Label 10100 6100 0    50   ~ 0
-CDI
-Text Label 10100 6300 0    50   ~ 0
-C~CS~
-Text Label 10100 6200 0    50   ~ 0
-CDO
-Text Label 10100 6400 0    50   ~ 0
 CCK
-Text Label 9700 6100 2    50   ~ 0
-CDIr
 Wire Wire Line
 	9100 6100 9100 6200
@@
 Wire Wire Line
 	7900 6400 7800 6400
-Wire Wire Line
-	5900 6200 5900 6300
-Connection ~ 5900 6200
 NoConn ~ 7450 2700
 NoConn ~ 7450 2900
 NoConn ~ 7450 3000
 NoConn ~ 7450 3100
+Text Label 5500 6200 2    50   ~ 0
+C~RST~
+$Comp
+L Device:R_Small R1
+U 1 1 687E63CA
+P 5600 6200
+F 0 "R1" V 5450 6200 50  0000 C CNN
+F 1 "33" V 5550 6200 50  0000 C BNN
+F 2 "stdpads:R_0603" H 5600 6200 50  0001 C CNN
+F 3 "~" H 5600 6200 50  0001 C CNN
+	1    5600 6200
+	0    1    1    0
+$EndComp
+$Comp
+L Device:R_Small R4
+U 1 1 687E7527
+P 5600 6450
+F 0 "R4" V 5450 6450 50  0000 C CNN
+F 1 "33" V 5550 6450 50  0000 C BNN
+F 2 "stdpads:R_0603" H 5600 6450 50  0001 C CNN
+F 3 "~" H 5600 6450 50  0001 C CNN
+	1    5600 6450
+	0    1    1    0
+$EndComp
+$Comp
+L Device:R_Small R5
+U 1 1 687E7710
+P 5600 6700
+F 0 "R5" V 5450 6700 50  0000 C CNN
+F 1 "33" V 5550 6700 50  0000 C BNN
+F 2 "stdpads:R_0603" H 5600 6700 50  0001 C CNN
+F 3 "~" H 5600 6700 50  0001 C CNN
+	1    5600 6700
+	0    1    1    0
+$EndComp
+$Comp
+L power:+3V3 #PWR0153
+U 1 1 6140B25C
+P 5800 6200
+F 0 "#PWR0153" H 5800 6050 50  0001 C CNN
+F 1 "+3V3" H 5800 6350 50  0000 C CNN
+F 2 "" H 5800 6200 50  0001 C CNN
+F 3 "" H 5800 6200 50  0001 C CNN
+	1    5800 6200
+	1    0    0    -1
+$EndComp
+Wire Wire Line
+	5700 6200 5800 6200
+Connection ~ 5800 6200
+Wire Wire Line
+	5800 6450 5700 6450
+Wire Wire Line
+	5800 6200 5800 6450
+Wire Wire Line
+	5800 6700 5700 6700
+$Comp
+L Device:R_Small R2
+U 1 1 6880B9BD
+P 9800 6400
+F 0 "R2" V 9650 6400 50  0000 C CNN
+F 1 "33" V 9750 6400 50  0000 C BNN
+F 2 "stdpads:R_0603" H 9800 6400 50  0001 C CNN
+F 3 "~" H 9800 6400 50  0001 C CNN
+	1    9800 6400
+	0    1    1    0
+$EndComp
+$Comp
+L Device:R_Small R6
+U 1 1 6881D7E4
+P 5600 6950
+F 0 "R6" V 5450 6950 50  0000 C CNN
+F 1 "33" V 5550 6950 50  0000 C BNN
+F 2 "stdpads:R_0603" H 5600 6950 50  0001 C CNN
+F 3 "~" H 5600 6950 50  0001 C CNN
+	1    5600 6950
+	0    1    1    0
+$EndComp
+Connection ~ 5800 6450
+Connection ~ 5800 6700
+Wire Wire Line
+	5800 6450 5800 6700
+Wire Wire Line
+	5800 6950 5700 6950
+Wire Wire Line
+	5800 6700 5800 6950
 $EndSCHEMATC

Commit message: Generated gerbers and documenation PDFs
Parts:
- removed RN1, RN2, RN3, RN4, RN5: 4x33, stdpads:R4_0402, symbol Device:R_Pack04
- added C35: 15p, stdpads:C_0603, symbol Device:C_Small
- added D1: White, stdpads:LED_0805, symbol Device:LED_Small_ALT
- added R10, R8, R9: 47, stdpads:R_0603, symbol Device:R_Small
- added R7: 180, stdpads:R_0805, symbol Device:R_Small
- J1: value Memory Expansion -> IIgs RAM Exp.
- R1, R4, R5, R6: value 33 -> 10k; LCSC Part (none) -> C25804; Mfg. Part Numbers (none) -> Uniroyal 0603WAF1002T5E; Notes (none) -> Any manufacturer's part is acceptable.
- R2: value 33 -> 47; LCSC Part (none) -> C23182; Mfg. Part Numbers (none) -> Uniroyal 0603WAF470JT5E; Notes (none) -> Any manufacturer's part is acceptable.
- R3: value 100 -> 47; footprint stdpads:R_0805 -> stdpads:R_0603; LCSC Part C17408 -> C23182; Mfg. Part Numbers Uniroyal 0805W8F1000T5E -> Uniroyal 0603WAF470JT5E
- U10, U9: Notes (none) -> Most 74LVC1G04 or 74AHC1G04 in SOT-353 package is acceptabl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
- U11: Notes (none) -> Most 1.2V regulator in SOT-23-5 package is acceptable.
- U12: Notes Most SPI flash in SOIC-8 (3.9mm / 150 mil width) package is acceptale. -> Most SPI flash in SOIC-8 (3.9mm / 150 mil width) package is acceptable.
- U13: Notes (none) -> Most 2.5V regulator in SOT-23-5 package is acceptable.
- U2: Notes Most 166 MHz 128/256 Mbit SDRAM is acceptable. -> Most 166 MHz 128/256 Mbit x16 SDRAM is acceptable.
- U4: Mfg. Part Numbers NXP 74AHCT245PW, TI SN74AHCT245PW -> NXP 74AHCT245PW, NXP 74AHCT245APW, TI SN74AHCT245PW,; Notes (none) -> Most 74AHCT245 in TSSOP-20 package is acceptable.
- U5, U6, U7: Mfg. Part Numbers NXP 74LVC245APW, TI SN74LVC245APW -> NXP 74LVC245APW, TI SN74LVC245APW, NXP 74AHC245PW, NXP 74AH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; Notes (none) -> Most 74LVC245 or 74AHC245 in TSSOP-20 package is acceptable.
Connections:
- net RD0r is gone; now on net RD0: U1.85 (IOT_80)
- net RD1r is gone; now on net RD1: U1.99 (IOT_93)
- net RD2r is gone; now on net RD3: U1.100 (IOT_95)
- net RD3r is gone; now on net RD2: U1.86 (IOT_81)
- net RD4r is gone; now on net RD5: U1.89 (IOT_84_GBIN1)
- net RD5r is gone; now on net RD4: U1.87 (IOT_82)
- net RD6r is gone; now on net RD6: U1.90 (IOT_85_GBIN0)
- net RD7r is gone; now on net RD7: U1.91 (IOT_86)
- net +3V3: now also R7.2
- net AClk: now also R9.2
- net Ain3: now also U7.14 (B4)
- net Ain4: now also U7.15 (B3)
- net Ain5: now also U7.16 (B2)
- net Ain6: now also U7.13 (B5)
- net Ain7: now also U7.17 (B1)
- net Ain8: now also U7.12 (B6)
- net Ain9: now also U7.11 (B7)
- net CCK: now also C35.1, R10.2; no longer J2.1 (Pin_1)
- net GND: now also C35.2
- net RClk: now also R8.2
- net ~CRAS~in: now also R3.1
- net at U4.19 (~OE~): now also U9.4 (Y); no longer R3.2
- net at U7.18 (B0): now also R3.2
- net at U10.4 (Y): now also R8.1, R9.1
- net LED: now reaches U1.82 (IOT_78)
- net LED: now also D1.1 (K)
- new net: D1.2 (A), R7.1
- new net CCKr2: J2.1 (Pin_1), R10.1
- no-connect marks 14 -> 9
Other:
- moved on the sheet: R2
